File: projects/cec-wifi-bridge-rev-a/cec-wifi-bridge-rev-a.brd (EAGLE design)
At the start: 76.2 x 25.4 mm, 15 parts, among them J1 DX4R005H91R1500, U1 MCP73831/2/OT, U2 TPS61200DRC

Commit message: Starting to add in the main bits.
Parts:
- added C6, C7: 14pF, passives:C0402
- added U3: ESP8266EX, espressif:ESP8266EX
- added X1: 26MHz, crystals:EPSON-TSX-3225
Connections:
- new net N$11: C6.1, U3.XTAL_IN, X1.P$3
- new net N$12: C7.2, U3.XTAL_OUT, X1.P$1
- net AGND: now also C6.2, C7.1, U3.GND, X1.P$2, X1.P$4
Changed lines of the file:
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@@
 <element name="U1" library="microchip" package="5-SOT23" value="MCP73831/2/OT" x="-38.1" y="12.7"/>
 <element name="U2" library="texas-instruments" package="S-PVSON-N10-DRC" value="TPS61200DRC" x="-22.86" y="12.7"/>
+<element name="U3" library="espressif" package="ESP8266EX" value="ESP8266EX" x="-45.72" y="3.81"/>
+<element name="X1" library="crystals" package="EPSON-TSX-3225" value="26MHz" x="-54.61" y="2.54"/>
+<element name="C6" library="passives" package="C0402" value="14pF" x="-55.88" y="-5.08"/>
+<element name="C7" library="passives" package="C0402" value="14pF" x="-55.88" y="-10.16"/>
 </elements>
 <signals>
@@
 <contactref element="J1" pad="P$5"/>
 <contactref element="J2" pad="2"/>
+<contactref element="C6" pad="2"/>
+<contactref element="C7" pad="1"/>
+<contactref element="X1" pad="P$2"/>
+<contactref element="X1" pad="P$4"/>
+<contactref element="U3" pad="GND"/>
+<wire x1="-55.4" y1="-5.08" x2="-56.36" y2="-10.16" width="0" layer="19" extent="1-1"/>
+<wire x1="-53.51" y1="1.74" x2="-55.4" y2="-5.08" width="0" layer="19" extent="1-1"/>
+<wire x1="-55.71" y1="3.34" x2="-53.51" y2="1.74" width="0" layer="19" extent="1-1"/>
+<wire x1="-45.72" y1="3.81" x2="-53.51" y2="1.74" width="0" layer="19" extent="1-1"/>
+<wire x1="-38.1" y1="11.3" x2="-45.72" y2="3.81" width="0" layer="19" extent="1-1"/>
 <wire x1="-32.12" y1="20.32" x2="-38.1" y2="11.3" width="0" layer="19" extent="1-1"/>
 <wire x1="-27.04" y1="20.32" x2="-32.12" y2="20.32" width="0" layer="19" extent="1-1"/>
@@
 <wire x1="-17.185" y1="20.32" x2="-22.86" y2="11.225" width="0" layer="19" extent="1-1"/>
 </signal>
+<signal name="N$11">
+<contactref element="U3" pad="XTAL_IN"/>
+<contactref element="X1" pad="P$3"/>
+<contactref element="C6" pad="1"/>
+<wire x1="-53.51" y1="3.34" x2="-56.36" y2="-5.08" width="0" layer="19" extent="1-1"/>
+<wire x1="-45.47" y1="6.21" x2="-53.51" y2="3.34" width="0" layer="19" extent="1-1"/>
+</signal>
+<signal name="N$12">
+<contactref element="U3" pad="XTAL_OUT"/>
+<contactref element="X1" pad="P$1"/>
+<contactref element="C7" pad="2"/>
+<wire x1="-55.71" y1="1.74" x2="-55.4" y2="-10.16" width="0" layer="19" extent="1-1"/>
+<wire x1="-44.97" y1="6.21" x2="-55.71" y2="1.74" width="0" layer="19" extent="1-1"/>
+</signal>
 </signals>

Commit message: Start wiring up the ESP8266.
Parts:
- added J3: DEBUG, pin-headers:2X04
- added J4: PROGRAM, pin-headers:1X03
- added R5: 12K, passives:R0402
- added R6, R7: 10K, passives:R0402
- added S1: RESET, switches:ALPS-SKQG
- added S2: UPLOAD, switches:ALPS-SKQG
- added U4: SPI-FLASH-SOIC8, flash:SOIC-8
- R1: value 20K -> 2K
- moved R1 36.4 mm to (-53.3, 15.2)
- moved R2 36.4 mm to (-57.1, 15.2)
- moved R3 36.4 mm to (-48.3, 15.2)
Connections:
- new net !RST: J3.1, R7.1, S1.P$3, S1.P$4, U3.EXT_RSTB, U3.XPD_DCDC
- new net FLASH_BOOT: R6.1, S2.P$1, S2.P$2, U3.GPIO0
- new net N$10: R5.2, U3.RES12K
- new net N$13: J4.1, U3.U0RXD
- new net N$14: J4.2, U3.U0TXD
- new net N$16: J3.2, U3.MTDO
- new net N$17: J3.4, U3.MTCK
- new net N$18: J3.6, U3.MTDI
- new net N$19: J3.8, U3.MTMS
- new net N$20: U3.SD_CLK, U4.P$6
- new net N$21: U3.SD_CMD, U4.P$1
- new net N$22: U3.SD_DATA_1, U4.P$5
- new net N$23: U4.P$2
- new net N$24: U3.SD_DATA_3, U4.P$3
- new net N$25: U3.SD_DATA_2, U4.P$7
- net +3V3: now also R6.2, R7.2, U3.CHIP_EN, U3.GPIO2, U3.VDD3P3, U3.VDD3P3$2, U3.VDDA, U3.VDDA$2, U3.VDDD, U3.VDDPST, U3.VDDPST$2, U3.VDD_RTC, U4.P$8
- net AGND: now also J3.5, J3.7, R5.1, S1.P$1, S1.P$2, S2.P$3, S2.P$4, U4.P$4

Commit message: Lots of tweaks and changes.
Parts:
- removed J4: PROGRAM, pin-headers:1X03
- added ANT1: INVERTED_F_ANTENNA+0, antenna:DN007+0
- added C10, C11, C12, C13, C14, C15, C16, C9: 0.1uF, passives:C0402
- added C8: 5.6pF, passives:C0402
- added J5: PROGRAM, pin-headers:1X05
- R4: value 820 -> 330
- moved R5 106.9 mm to (47.0, 14.0)
- moved U4 104.5 mm to (34.3, 25.4), turned to 270 degrees
- moved C6 101.5 mm to (44.5, 10.2)
- moved X1 95.6 mm to (40.6, 10.2)
- moved C7 93.7 mm to (35.6, 10.2)
- moved U3 88.7 mm to (41.9, 17.8), turned to 180 degrees
- moved J3 64.4 mm to (-26.7, -58.4)
- moved U1 54.7 mm to (16.5, 16.5)
- moved S1 50.6 mm to (27.9, 3.81)
- moved S2 49.4 mm to (16.5, 3.81)
- moved J2 47.4 mm to (25.4, 27.9)
- moved U2 46.0 mm to (22.9, 17.8)
- moved R1 35.9 mm to (-17.8, 10.2)
- moved R2 35.9 mm to (-21.6, 10.2)
- moved R3 35.9 mm to (-12.7, 10.2)
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Connections:
- net N$17 renamed TCK
- net N$3 renamed VBUS
- removed net N$13: J4.1, U3.U0RXD
- removed net N$14: J4.2, U3.U0TXD
- removed net N$16: J3.2, U3.MTDO
- removed net N$18: J3.6, U3.MTDI
- removed net N$19: J3.8, U3.MTMS
- new net ANT: C8.1, U3.LNA
- new net CEC_IN: U3.GPIO4
- new net CEC_OUT: U3.GPOIO5
- new net N$26: ANT1.FEED, C8.2
- new net TDI: J3.8, U3.MTDI
- new net TDO: J3.6, U3.MTDO
- new net TMS: J3.2, U3.MTMS
- new net UART_RX: J5.1, U3.U0RXD
- new net UART_TX: J5.2, U3.U0TXD
- net +3V3: now also C10.1, C11.1, C12.1, C13.1, C14.1, C15.1, C16.1, C9.1; no longer U3.VDD_RTC
- net AGND: now also ANT1.GND, ANT1.GND@1, C10.2, C11.2, C12.2, C13.2, C14.2, C15.2, C16.2, C9.2, J5.5
Other:
- board size 76.2 x 25.4 mm -> 76.2 x 30.5 mm

Commit message: Lots of board layout work.
The board is basically done.

It has a real shape now, things are laid out.  We have fiducials,
alignment holes, rounded edges, the PCB antenna with the proper
setbacks, ground plane stitching, we have our logo in place (!), and
things are generally buttoned up.

We still need to fill out the BOM entirely, as well as clean up the
schematic sheets and add proper titles/descriptions, etc.

Also need to look into bitmap art for open source hardware to start
throwing on the board.  Should probably add the license / attribution
stuff, as well.
Parts:
- added C17: 27pF, passives:C0402
- added C18: 0.1uF, passives:C0402
- added D2: 1N4148, diodes:SOD123
- added J4: 10029449-001RLF, amphenol:10029449
- added R10, R15: 47K, passives:R0402
- added R11, R8: 220, passives:R0402
- added R12: 100K, passives:R0402
- added R13: 27K, passives:R0402
- added R14: 1M, passives:R0402
- added R9: 470K, passives:R0402
- added T1, T2: MMBT3904, transistors:SC-70
- added U$1, U$2, U$3: FIDUCIAL-1MM, fiducials:FIDUCIAL_1MM
- moved C16 128.9 mm to (48.6, 25.5)
- moved J3 118.4 mm to (57.3, 25.0), turned to 90 degrees
- moved J5 100.2 mm to (35.7, 10.0), turned to 270 degrees
- moved C14 99.3 mm to (48.6, 23.1)
- moved C15 96.1 mm to (44.8, 17.8)
- moved C12 94.2 mm to (48.6, 24.4)
- moved C11 90.5 mm to (45.2, 27.9)
- moved C10 85.9 mm to (42.7, 28.4), turned to 90 degrees
- moved C9 85.4 mm to (48.6, 20.7)
- moved C13 80.3 mm to (32.0, 18.7), turned to 180 degrees
- moved R7 72.2 mm to (51.3, 13.2)
- moved R6 66.3 mm to (54.2, 13.2), turned to 180 degrees
- moved C4 57.6 mm to (25.1, 8.00)
- moved C5 51.9 mm to (26.0, 9.78)
- moved C2 50.1 mm to (22.2, 3.81), turned to 270 degrees
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Connections:
- removed net CEC_IN: U3.GPIO4
- removed net CEC_OUT: U3.GPOIO5
- removed net N$5: R3.1
- new net CEC_RX: R12.1, T1.P$3, U3.GPOIO5
- new net CEC_TX: R15.1, U3.GPIO4
- new net HDMI_CEC: C17.1, D2.C, J4.P$13, R14.2, T2.P$3
- new net N$15: R8.2, T1.P$2
- new net N$16: R14.1, R9.2, T1.P$1
- new net N$18: D2.A, R13.2
- new net N$27: R11.2, T2.P$2
- new net N$3: C17.2, R10.2, R15.2, T2.P$1
- net +3V3: now also C18.1, R12.2, R13.1
- net AGND: now also C18.2, J4.P$17, R10.1, R11.1, R3.1, R8.1, R9.1, U3.P$1, U3.P$2, U3.P$3, U3.P$4, U3.P$5, U3.P$6, U3.P$7, U3.P$8, U3.P$9
Routing:
- net FLASH_BOOT: track 0.00 -> 43.7 mm, vias 0 -> 2
- net !RST: track 0.00 -> 43.4 mm, vias 0 -> 3
- net +3V3: track 0.00 -> 39.6 mm, vias 0 -> 14
- net N$1: track 0.00 -> 33.6 mm, vias 0 -> 3
- net TCK: track 0.00 -> 30.8 mm, vias 0 -> 2
- net CEC_RX: track 0.00 -> 22.8 mm
- net ANT: track 0.00 -> 21.2 mm
- net N$24: track 0.00 -> 20.2 mm
- net HDMI_CEC: track 0.00 -> 18.7 mm
- net N$22: track 0.00 -> 18.4 mm
- net CEC_TX: track 0.00 -> 18.3 mm
- net TDI: track 0.00 -> 18.3 mm
- net TDO: track 0.00 -> 17.4 mm
- net N$25: track 0.00 -> 15.7 mm
- net TMS: track 0.00 -> 14.6 mm
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- added copper zone on layer 15, net +3V3
- added copper zone on layer 1, net AGND
- added copper zone on layer 2, net AGND
- added copper zone on layer 1, net N$1
- added copper zone on layer 1, net N$9
Other:
- board size 76.2 x 30.5 mm -> 75.9 x 32.4 mm
- board text added: "BAT"
- board text added: "WiFi-CEC Bridge rev A Nuclear Furnace, 2017"

Commit message: cleanup
Connections:
- net N$23: now also U3.SD_DATA_0
Routing:
- net N$23: track 0.00 -> 6.74 mm, vias 0 -> 2
Changed lines of the file:
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@@
 <layer number="25" name="tNames" color="7" fill="1" visible="yes" active="yes"/>
 <layer number="26" name="bNames" color="7" fill="1" visible="yes" active="yes"/>
-<layer number="27" name="tValues" color="7" fill="1" visible="yes" active="yes"/>
-<layer number="28" name="bValues" color="7" fill="1" visible="yes" active="yes"/>
+<layer number="27" name="tValues" color="7" fill="1" visible="no" active="yes"/>
+<layer number="28" name="bValues" color="7" fill="1" visible="no" active="yes"/>
 <layer number="29" name="tStop" color="7" fill="3" visible="no" active="yes"/>
 <layer number="30" name="bStop" color="7" fill="6" visible="no" active="yes"/>
@@
 <element name="J2" library="pin-headers" package="1X02" value="" x="30.226" y="5.461" smashed="yes" rot="R270">
 <attribute name="VALUE" x="27.051" y="8.001" size="1.27" layer="27" rot="R270"/>
+<attribute name="BOM" value="EXCLUDE" x="30.226" y="5.461" size="1.778" layer="27" rot="R270" display="off"/>
 </element>
 <element name="L1" library="passives" package="COILCRAFT-XPL2010" value="2.2uH" x="21.082" y="11.049" smashed="yes" rot="R180">
@@
 <attribute name="NAME" x="30.734" y="25.908" size="1.27" layer="25"/>
 </element>
-<element name="ANT1" library="antenna" package="DN007+0" value="INVERTED_F_ANTENNA+0" x="69.85" y="20.193" rot="R270"/>
+<element name="ANT1" library="antenna" package="DN007+0" value="INVERTED_F_ANTENNA+0" x="69.85" y="20.193" rot="R270">
+<attribute name="BOM" value="EXCLUDE" x="69.85" y="20.193" size="1.778" layer="27" rot="R270" display="off"/>
+</element>
 <element name="C8" library="passives" package="C0402" value="5.6pF" x="65.786" y="17.907" smashed="yes">
 <attribute name="NAME" x="67.056" y="17.399" size="1.27" layer="25"/>
@@
 <wire x1="50.828" y1="13.208" x2="50.828" y2="7.335" width="0.1524" layer="1"/>
 <wire x1="50.828" y1="7.335" x2="51.106" y2="7.057" width="0.254" layer="1"/>
-<wire x1="45.72" y1="20.828" x2="50.673" y2="15.875" width="0.1524" layer="16"/>
+<wire x1="45.707" y1="20.841" x2="50.673" y2="15.875" width="0.1524" layer="16"/>
 <wire x1="50.673" y1="15.875" x2="50.673" y2="14.351" width="0.1524" layer="16"/>
 <via x="50.673" y="14.351" extent="1-16" drill="0.254"/>
@@
 <wire x1="50.673" y1="13.363" x2="50.828" y2="13.208" width="0.1524" layer="1"/>
 <wire x1="45.707" y1="20.841" x2="45.184" y2="20.841" width="0.1524" layer="1"/>
-<wire x1="45.72" y1="20.828" x2="45.707" y2="20.841" width="0" layer="19" extent="16-16"/>
 </signal>
 <signal name="TDO">
@@
 <signal name="N$23">
 <contactref element="U4" pad="P$2"/>
+<contactref element="U3" pad="SD_DATA_0"/>
+<wire x1="37.325" y1="21.844" x2="35.941" y2="21.844" width="0.1524" layer="1"/>
+<via x="35.941" y="21.844" extent="1-16" drill="0.254"/>
+<wire x1="35.941" y1="21.844" x2="39.116" y2="21.844" width="0.1524" layer="16"/>
+<wire x1="39.116" y1="21.844" x2="39.751" y2="22.479" width="0.1524" layer="16"/>
+<via x="39.751" y="22.479" extent="1-16" drill="0.254"/>
+<wire x1="39.751" y1="22.479" x2="41.022" y2="22.479" width="0.1524" layer="1"/>
+<wire x1="41.022" y1="22.479" x2="41.034" y2="22.491" width="0.1524" layer="1"/>
 </signal>
 <signal name="N$24">

Commit message: Filled in BOM and super stitched.
Filled in all of the BOM values.  Also stitches the hell out of the
board.  Realllly stitched it.  Probably overstitched it.
Parts:
- R3: value 198K -> 196K
- moved J3 3.68 mm to (57.3, 28.7)
- moved ANT1 3.68 mm to (69.8, 23.9)
- moved C10 3.68 mm to (42.7, 32.1)
- moved C11 3.68 mm to (45.2, 31.6)
- moved C12 3.68 mm to (48.6, 28.1)
- moved C13 3.68 mm to (32.0, 22.4)
- moved C14 3.68 mm to (48.6, 26.8)
- moved C15 3.68 mm to (44.8, 21.5)
- moved C16 3.68 mm to (48.6, 29.2)
- moved C17 3.68 mm to (24.8, 27.3)
- moved C18 3.68 mm to (38.6, 30.6)
- moved C6 3.68 mm to (45.8, 18.7)
- moved C7 3.68 mm to (39.4, 18.7)
- moved C8 3.68 mm to (65.8, 21.6)
- moved C9 3.68 mm to (48.6, 24.4)
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Routing:
- net FLASH_BOOT: track 43.7 -> 47.4 mm
- net UART_TX: track 12.7 -> 16.4 mm
- net UART_RX: track 9.85 -> 13.5 mm
- net !RST: track 43.4 -> 47.1 mm
- net AGND: vias 301 -> 534
Other:
- board size 75.9 x 32.4 mm -> 75.9 x 36.1 mm
- board text added: "+"

Commit message: Add BOM parts and adjust alignment holes.
Added the remaining two BOM values.

Adjusted the location of the alignment pin holes so that we can cleanly
fit the LiPo battery on the underside of the board without it being
under the PCB antenna and without it being too close to the HDMI
through-hole pins.
Parts:
- moved C14 0.25 mm to (48.6, 27.1)
- moved C12 0.13 mm to (48.6, 28.2)
- moved C16 0.13 mm to (48.6, 29.3)
Routing:
- net AGND: vias 534 -> 547

Commit message: Add LED and more board tweaking.
Added another LED after realizing that STAT on the battery charger IC is
actually tri-state -- thanks, Adafruit!  This means we can now show when
the battery is charging and when it's full, wee!

Also moved bits and pieces around on the board.  Spread out the
stitching vias, moved vias out of the way of the silkscreen, etc etc.
Parts:
- added D3: 3.2V, 5mA, dialight:DIALIGHT-0603
- added R16: 330, passives:R0603
- D1: value 2V, 4mA -> 2V, 5mA
- R4: device passives:R0805 -> passives:R0603
- moved D1 18.1 mm to (23.1, 16.0)
- moved R4 17.9 mm to (26.8, 16.0)
- moved U$2 2.84 mm to (51.6, 19.7)
Connections:
- new net N$5: D3.1, R16.1
- net AGND: now also D3.2
- net N$7: now also R16.2
Routing:
- net N$7: track 2.13 -> 24.1 mm, vias 0 -> 2
- net VBUS: track 11.6 -> 24.5 mm, vias 0 -> 2
- net N$5: track 0.00 -> 4.47 mm
- net AGND: vias 547 -> 565
Other:
- board text added: "CHRG"
- board text added: "FULL"
