File: projects/cec-wifi-bridge-rev-a/cec-wifi-bridge-rev-a.brd (EAGLE design)
At the start: 75.9 x 36.1 mm, 56 parts, among them J1 DX4R005H91R1500, J3 DEBUG, J4 10029449-001RLF, J5 PROGRAM, T1 MMBT3904, T2 MMBT3904, U1 MCP73831/2/OT, U2 TPS61200DRC, U3 ESP8266EX, U4 SPI-FLASH-SOIC8, X1 26MHz

Commit message: Switch to DX4R005HJ5R2000 for USB connector.
The other version we were using had no 3D model available from JAE, so I
found one that did, so we can properly design the enclosure and model it
all assembled.
Parts:
- J1: value DX4R005H91R1500 -> DX4R005HJ5R2000; device jae:DX4R005H91R1500 -> jae:DX4R005HJ5R2000
- moved J1 1.40 mm to (1.52, 7.11)
Connections:
- net AGND: now also J1.5, J1.CASE_1, J1.CASE_2, J1.CASE_3, J1.CASE_4; no longer J1.P$5
- net VBUS: now also J1.1; no longer J1.P$1
Routing:
- net AGND: vias 565 -> 567
Changed lines of the file:
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@@
 <layer number="27" name="tValues" color="7" fill="1" visible="no" active="yes"/>
 <layer number="28" name="bValues" color="7" fill="1" visible="no" active="yes"/>
-<layer number="29" name="tStop" color="7" fill="3" visible="no" active="yes"/>
-<layer number="30" name="bStop" color="7" fill="6" visible="no" active="yes"/>
-<layer number="31" name="tCream" color="7" fill="4" visible="no" active="yes"/>
-<layer number="32" name="bCream" color="7" fill="5" visible="no" active="yes"/>
+<layer number="29" name="tStop" color="7" fill="3" visible="yes" active="yes"/>
+<layer number="30" name="bStop" color="7" fill="6" visible="yes" active="yes"/>
+<layer number="31" name="tCream" color="7" fill="4" visible="yes" active="yes"/>
+<layer number="32" name="bCream" color="7" fill="5" visible="yes" active="yes"/>
 <layer number="33" name="tFinish" color="6" fill="3" visible="no" active="yes"/>
 <layer number="34" name="bFinish" color="6" fill="6" visible="no" active="yes"/>
@@
 <elements>
 <element name="C1" library="passives" package="C0603" value="4.7uF" x="16.002" y="7.366" smashed="yes" rot="R270">
-<attribute name="NAME" x="15.367" y="4.953" size="1.27" layer="25" font="vector" rot="R270"/>
+<attribute name="NAME" x="15.367" y="11.557" size="1.27" layer="25" font="vector" rot="R270"/>
 <attribute name="PN" value="GRM188R61A475KE15D" x="16.002" y="7.366" size="1.778" layer="27" rot="R270" display="off"/>
 </element>
@@
 <attribute name="PN" value="598-8020-107F" x="23.114" y="16.002" size="1.778" layer="27" display="off"/>
 </element>
-<element name="J1" library="jae" package="DX4R005H91R1500" value="DX4R005H91R1500" x="0.127" y="7.112" smashed="yes" rot="R270">
-<attribute name="NAME" x="5.222" y="4.766" size="1.27" layer="25" font="vector" rot="R270"/>
-<attribute name="PN" value="DX4R005H91R1500" x="0.127" y="7.112" size="1.778" layer="27" rot="R270" display="off"/>
+<element name="J1" library="jae" package="DX4R005HJ5R2000" value="DX4R005HJ5R2000" x="1.524" y="7.112" smashed="yes" rot="R270">
+<attribute name="NAME" x="6.365" y="4.766" size="1.27" layer="25" font="vector" rot="R270"/>
+<attribute name="PN" value="DX4R005HJ5R2000" x="1.524" y="7.112" size="1.778" layer="27" rot="R270" display="off"/>
 </element>
 <element name="J2" library="pin-headers" package="1X02" value="" x="30.226" y="5.461" smashed="yes" rot="R270">
@@
 <contactref element="C3" pad="2"/>
 <contactref element="C2" pad="2"/>
-<contactref element="J1" pad="P$5"/>
+<contactref element="J1" pad="5"/>
 <contactref element="J2" pad="2"/>
 <contactref element="C6" pad="2"/>
@@
 <via x="31.75" y="15.113" extent="1-16" drill="0.254"/>
 <via x="31.75" y="10.033" extent="1-16" drill="0.254"/>
-<via x="5.715" y="10.033" extent="1-16" drill="0.254"/>
-<via x="5.588" y="4.953" extent="1-16" drill="0.254"/>
+<via x="5.334" y="10.922" extent="1-16" drill="0.254"/>
+<via x="5.334" y="3.302" extent="1-16" drill="0.254"/>
 <via x="12.7" y="10.033" extent="1-16" drill="0.254"/>
 <via x="28.321" y="5.461" extent="1-16" drill="0.254"/>
@@
 <via x="1.27" y="16.891" extent="1-16" drill="0.254"/>
 <via x="2.794" y="13.208" extent="1-16" drill="0.254"/>
-<via x="2.54" y="10.668" extent="1-16" drill="0.254"/>
-<via x="2.54" y="9.398" extent="1-16" drill="0.254"/>
-<via x="1.27" y="8.128" extent="1-16" drill="0.254"/>
-<via x="1.27" y="6.858" extent="1-16" drill="0.254"/>
-<via x="1.27" y="5.588" extent="1-16" drill="0.254"/>
-<via x="2.54" y="4.318" extent="1-16" drill="0.254"/>
+<via x="1.27" y="7.112" extent="1-16" drill="0.254"/>
 <via x="2.54" y="3.048" extent="1-16" drill="0.254"/>
 <via x="2.54" y="1.778" extent="1-16" drill="0.254"/>
@@
 <via x="14.097" y="2.921" extent="1-16" drill="0.254"/>
 <via x="13.716" y="4.191" extent="1-16" drill="0.254"/>
-<via x="6.604" y="3.302" extent="1-16" drill="0.254"/>
-<via x="2.54" y="7.62" extent="1-16" drill="0.254"/>
-<via x="2.54" y="6.096" extent="1-16" drill="0.254"/>
+<via x="6.985" y="4.572" extent="1-16" drill="0.254"/>
+<via x="2.54" y="7.112" extent="1-16" drill="0.254"/>
 <via x="8.001" y="9.398" extent="1-16" drill="0.254"/>
 <via x="32.258" y="7.747" extent="1-16" drill="0.254"/>
@@
 <via x="25.019" y="14.859" extent="1-16" drill="0.254"/>
 <via x="23.241" y="14.859" extent="1-16" drill="0.254"/>
-<via x="9.144" y="5.08" extent="1-16" drill="0.254"/>
-<via x="7.747" y="4.572" extent="1-16" drill="0.254"/>
+<via x="9.398" y="5.08" extent="1-16" drill="0.254"/>
+<via x="8.128" y="5.08" extent="1-16" drill="0.254"/>
 <via x="7.239" y="7.239" extent="1-16" drill="0.254"/>
-<via x="6.985" y="5.588" extent="1-16" drill="0.254"/>
+<via x="7.239" y="5.969" extent="1-16" drill="0.254"/>
 <via x="12.446" y="3.429" extent="1-16" drill="0.254"/>
-<via x="7.874" y="3.048" extent="1-16" drill="0.254"/>
+<via x="8.128" y="3.429" extent="1-16" drill="0.254"/>
 <via x="10.795" y="2.921" extent="1-16" drill="0.254"/>
 <via x="10.922" y="4.572" extent="1-16" drill="0.254"/>
@@
 <via x="15.367" y="12.7" extent="1-16" drill="0.254"/>
 <via x="13.716" y="11.684" extent="1-16" drill="0.254"/>
+<contactref element="J1" pad="CASE_1"/>
+<contactref element="J1" pad="CASE_2"/>
+<contactref element="J1" pad="CASE_3"/>
+<contactref element="J1" pad="CASE_4"/>
+<via x="1.27" y="11.684" extent="1-16" drill="0.254"/>
+<via x="2.794" y="11.811" extent="1-16" drill="0.254"/>
+<via x="3.175" y="9.525" extent="1-16" drill="0.254"/>
+<via x="3.175" y="4.699" extent="1-16" drill="0.254"/>
+<via x="1.27" y="3.048" extent="1-16" drill="0.254"/>
+<via x="15.113" y="4.318" extent="1-16" drill="0.254"/>
+<via x="15.748" y="3.175" extent="1-16" drill="0.254"/>
+<via x="25.781" y="4.699" extent="1-16" drill="0.254"/>
 </signal>
 <signal name="N$4">
@@
 <contactref element="U1" pad="4"/>
 <contactref element="D1" pad="1"/>
-<contactref element="J1" pad="P$1"/>
-<wire x1="4.252" y1="8.412" x2="9.017" y2="8.412" width="0.4064" layer="1"/>
+<contactref element="J1" pad="1"/>
+<wire x1="4.099" y1="8.412" x2="9.017" y2="8.412" width="0.4064" layer="1"/>
 <wire x1="9.017" y1="8.412" x2="11.269" y2="8.412" width="0.4064" layer="1"/>
 <wire x1="11.269" y1="8.412" x2="11.3" y2="8.443" width="0.4064" layer="1"/>
