File: projects/cec-wifi-bridge-rev-a/cec-wifi-bridge-rev-a.brd (EAGLE design)
At the start: 75.9 x 36.1 mm, 56 parts, among them J1 DX4R005HJ5R2000, J3 DEBUG, J4 10029449-001RLF, J5 PROGRAM, T1 MMBT3904, T2 MMBT3904, U1 MCP73831/2/OT, U2 TPS61200DRC, U3 ESP8266EX, U4 SPI-FLASH-SOIC8, X1 26MHz

Commit message: More sane stitching.
The stitching before was haphazard, ugly, overkill, and generally
wasteful.  I did a more sane and uniform stitching of ground.

Looks better, and I'm guessing things will function just the same.
Routing:
- net AGND: vias 567 -> 387

Commit message: Fixing up the alignment of the USB port with the actuality of the enclosure.
Parts:
- moved J1 0.71 mm to (1.52, 6.40)
Routing:
- net AGND: vias 387 -> 389
Changed lines of the file:
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@@
 <attribute name="PN" value="598-8020-107F" x="23.114" y="16.002" size="1.778" layer="27" display="off"/>
 </element>
-<element name="J1" library="jae" package="DX4R005HJ5R2000" value="DX4R005HJ5R2000" x="1.524" y="7.112" smashed="yes" rot="R270">
-<attribute name="NAME" x="6.365" y="4.766" size="1.27" layer="25" font="vector" rot="R270"/>
-<attribute name="PN" value="DX4R005HJ5R2000" x="1.524" y="7.112" size="1.778" layer="27" rot="R270" display="off"/>
+<element name="J1" library="jae" package="DX4R005HJ5R2000" value="DX4R005HJ5R2000" x="1.524" y="6.4008" smashed="yes" rot="R270">
+<attribute name="NAME" x="6.365" y="4.0548" size="1.27" layer="25" font="vector" rot="R270"/>
+<attribute name="PN" value="DX4R005HJ5R2000" x="1.524" y="6.4008" size="1.778" layer="27" rot="R270" display="off"/>
 </element>
 <element name="J2" library="pin-headers" package="1X02" value="" x="30.226" y="5.461" smashed="yes" rot="R270">
@@
 <via x="1.27" y="18.161" extent="1-16" drill="0.254"/>
 <via x="1.27" y="16.891" extent="1-16" drill="0.254"/>
-<via x="1.27" y="7.112" extent="1-16" drill="0.254"/>
+<via x="1.27" y="6.477" extent="1-16" drill="0.254"/>
 <via x="2.54" y="1.778" extent="1-16" drill="0.254"/>
 <via x="3.81" y="1.778" extent="1-16" drill="0.254"/>
@@
 <via x="6.985" y="28.067" extent="1-16" drill="0.254"/>
 <via x="6.477" y="29.083" extent="1-16" drill="0.254"/>
-<via x="5.461" y="7.62" extent="1-16" drill="0.254"/>
-<via x="6.096" y="7.62" extent="1-16" drill="0.254"/>
-<via x="5.461" y="6.985" extent="1-16" drill="0.254"/>
-<via x="6.096" y="6.985" extent="1-16" drill="0.254"/>
-<via x="5.461" y="6.35" extent="1-16" drill="0.254"/>
-<via x="6.096" y="6.35" extent="1-16" drill="0.254"/>
+<via x="6.223" y="6.35" extent="1-16" drill="0.254"/>
+<via x="6.858" y="6.35" extent="1-16" drill="0.254"/>
+<via x="6.223" y="5.715" extent="1-16" drill="0.254"/>
+<via x="6.858" y="5.715" extent="1-16" drill="0.254"/>
+<via x="6.223" y="5.08" extent="1-16" drill="0.254"/>
+<via x="6.858" y="5.08" extent="1-16" drill="0.254"/>
 <via x="12.7" y="7.493" extent="1-16" drill="0.254"/>
 <via x="12.7" y="8.128" extent="1-16" drill="0.254"/>
@@
 <contactref element="J1" pad="CASE_4"/>
 <via x="1.27" y="11.684" extent="1-16" drill="0.254"/>
-<via x="1.27" y="3.048" extent="1-16" drill="0.254"/>
+<via x="1.397" y="2.413" extent="1-16" drill="0.254"/>
 <via x="63.5" y="32.131" extent="1-16" drill="0.254"/>
 <via x="63.5" y="29.591" extent="1-16" drill="0.254"/>
@@
 <via x="28.829" y="13.716" extent="1-16" drill="0.254"/>
 <via x="34.29" y="3.048" extent="1-16" drill="0.254"/>
+<via x="1.27" y="10.414" extent="1-16" drill="0.254"/>
+<via x="3.81" y="10.541" extent="1-16" drill="0.254"/>
 </signal>
 <signal name="N$4">
@@
 <contactref element="D1" pad="1"/>
 <contactref element="J1" pad="1"/>
-<wire x1="4.099" y1="8.412" x2="9.017" y2="8.412" width="0.4064" layer="1"/>
+<wire x1="4.099" y1="7.7008" x2="6.6848" y2="7.7008" width="0.4064" layer="1"/>
+<wire x1="6.6848" y1="7.7008" x2="7.396" y2="8.412" width="0.4064" layer="1"/>
 <wire x1="9.017" y1="8.412" x2="11.269" y2="8.412" width="0.4064" layer="1"/>
 <wire x1="11.269" y1="8.412" x2="11.3" y2="8.443" width="0.4064" layer="1"/>
@@
 <wire x1="9.017" y1="9.398" x2="9.017" y2="9.017" width="0.254" layer="1"/>
 <wire x1="9.017" y1="8.412" x2="9.017" y2="9.398" width="0.254" layer="1"/>
+<wire x1="9.017" y1="8.412" x2="7.396" y2="8.412" width="0.4064" layer="1"/>
 </signal>
 <signal name="N$7">

Commit message: Add testpoints for the power rails.
Parts:
- added TP1, TP2, TP3: TESTPOINT-WITH-GND, test:TESTPOINT-1.5-WITH-GND
Connections:
- removed net N$1: C1.1, C3.1, J2.1, L1.P$2, R2.2, U1.3, U2.P$5, U2.P$6, U2.P$8
- new net VBAT: C1.1, C3.1, J2.1, L1.P$2, R2.2, TP3.S, U1.3, U2.P$5, U2.P$6, U2.P$8
- net +3V3: now also TP2.S
- net AGND: now also TP1.G, TP2.G, TP3.G
- net VBUS: now also TP1.S
Routing:
- net VBAT: track 0.00 -> 37.5 mm, vias 0 -> 3
- net N$1: track 33.4 -> 0.00 mm, vias 3 -> 0
- net VBUS: track 24.9 -> 31.4 mm, vias 2 -> 3
- net +3V3: track 40.0 -> 41.9 mm, vias 14 -> 15
- net AGND: vias 389 -> 400
- added copper zone on layer 1, net VBAT
- removed copper zone on layer 1, net N$1
Other:
- board text added: "+3V3"
- board text added: "VBAT"
- board text added: "VBUS"
- board text removed: "BAT"
Changed lines of the file:
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@@
 <layer number="27" name="tValues" color="7" fill="1" visible="no" active="yes"/>
 <layer number="28" name="bValues" color="7" fill="1" visible="no" active="yes"/>
-<layer number="29" name="tStop" color="7" fill="3" visible="yes" active="yes"/>
-<layer number="30" name="bStop" color="7" fill="6" visible="yes" active="yes"/>
+<layer number="29" name="tStop" color="7" fill="3" visible="no" active="yes"/>
+<layer number="30" name="bStop" color="7" fill="6" visible="no" active="yes"/>
 <layer number="31" name="tCream" color="7" fill="4" visible="yes" active="yes"/>
 <layer number="32" name="bCream" color="7" fill="5" visible="yes" active="yes"/>
@@
 <wire x1="72.771" y1="36.068" x2="3.048" y2="36.068" width="0" layer="20"/>
 <wire x1="3.048" y1="36.068" x2="0" y2="32.893" width="0" layer="20" curve="90"/>
-<text x="33.401" y="2.794" size="1.27" layer="25" font="vector" ratio="12" rot="R90">BAT</text>
+<text x="33.401" y="2.921" size="1.27" layer="25" font="vector" ratio="12" rot="R90">VBAT</text>
 <text x="35.8902" y="21.5392" size="1.778" layer="26" font="vector" ratio="14" rot="MR0">WiFi-CEC Bridge
 rev A
@@
 <circle x="62.484" y="16.51" radius="3.683" width="0.0508" layer="51"/>
 <circle x="8.89" y="12.954" radius="3.683" width="0.0508" layer="51"/>
+<text x="16.383" y="4.064" size="1.27" layer="25" font="vector" ratio="12" rot="R180">VBUS</text>
+<text x="43.688" y="11.557" size="1.27" layer="25" font="vector" ratio="12">+3V3</text>
 </plain>
 <attributes>
@@
 </element>
 <element name="J1" library="jae" package="DX4R005HJ5R2000" value="DX4R005HJ5R2000" x="1.524" y="6.4008" smashed="yes" rot="R270">
-<attribute name="NAME" x="6.365" y="4.0548" size="1.27" layer="25" font="vector" rot="R270"/>
+<attribute name="NAME" x="6.111" y="10.2778" size="1.27" layer="25" font="vector" rot="R270"/>
 <attribute name="PN" value="DX4R005HJ5R2000" x="1.524" y="6.4008" size="1.778" layer="27" rot="R270" display="off"/>
 </element>
@@
 </element>
 <element name="S1" library="switches" package="ALPS-SKQG" value="RESET" x="48.006" y="5.207" smashed="yes" rot="R180">
-<attribute name="VALUE" x="43.942" y="8.255" size="1.27" layer="25" font="vector" ratio="12"/>
+<attribute name="VALUE" x="43.815" y="8.636" size="1.27" layer="25" font="vector" ratio="12"/>
 <attribute name="PN" value="SKQGAKE010" x="48.006" y="5.207" size="1.778" layer="27" rot="R180" display="off"/>
 </element>
@@
 </element>
 <element name="S2" library="switches" package="ALPS-SKQG" value="UPLOAD" x="57.658" y="5.207" smashed="yes">
-<attribute name="VALUE" x="53.594" y="8.255" size="1.27" layer="25" font="vector" ratio="12"/>
+<attribute name="VALUE" x="53.594" y="8.636" size="1.27" layer="25" font="vector" ratio="12"/>
 <attribute name="PN" value="SKQGAKE010" x="57.658" y="5.207" size="1.778" layer="27" display="off"/>
 </element>
@@
 </element>
 <element name="J5" library="pin-headers" package="1X05" value="PROGRAM" x="35.687" y="10.033" smashed="yes" rot="R270">
-<attribute name="VALUE" x="32.512" y="16.51" size="1.27" layer="25" font="vector" ratio="12" rot="R270"/>
+<attribute name="VALUE" x="37.592" y="10.414" size="1.27" layer="25" font="vector" ratio="12" rot="R270"/>
 <attribute name="PN" value="M20-9990546" x="35.687" y="10.033" size="1.778" layer="27" rot="R270" display="off"/>
 </element>
@@
 <attribute name="VALUE" x="21.463" y="18.796" size="1.27" layer="27"/>
 </element>
+<element name="TP1" library="test" package="TESTPOINT-1.5-WITH-GND" value="TESTPOINT-WITH-GND" x="9.017" y="3.429" smashed="yes">
+<attribute name="VALUE" x="6.731" y="4.953" size="1.27" layer="27"/>
+</element>
+<element name="TP2" library="test" package="TESTPOINT-1.5-WITH-GND" value="TESTPOINT-WITH-GND" x="41.021" y="12.192" smashed="yes">
+<attribute name="VALUE" x="38.735" y="13.716" size="1.27" layer="27"/>
+</element>
+<element name="TP3" library="test" package="TESTPOINT-1.5-WITH-GND" value="TESTPOINT-WITH-GND" x="32.385" y="10.16" smashed="yes" rot="R90">
+<attribute name="VALUE" x="30.861" y="7.874" size="1.27" layer="27" rot="R90"/>
+</element>
 </elements>
 <signals>
-<signal name="N$1">
+<signal name="VBAT">
 <contactref element="U2" pad="P$5"/>
 <contactref element="U1" pad="3"/>
@@
 <contactref element="C1" pad="1"/>
 <contactref element="L1" pad="P$2"/>
-<contactref element="J2" pad="1"/>
 <polygon width="0.254" layer="1" thermals="no">
 <vertex x="13.589" y="8.128"/>
@@
 <wire x1="19.685" y1="9.525" x2="19.177" y2="10.033" width="0.1524" layer="16"/>
 <via x="19.177" y="10.033" extent="1-16" drill="0.254"/>
-<wire x1="30.226" y1="6.731" x2="30.226" y2="10.541" width="1.016" layer="1"/>
 <wire x1="30.226" y1="10.541" x2="26.924" y2="13.843" width="1.016" layer="1"/>
 <wire x1="26.924" y1="13.843" x2="20.701" y2="13.843" width="1.016" layer="1"/>
@@
 <wire x1="19.05" y1="3.556" x2="19.05" y2="5.461" width="0.1524" layer="1"/>
 <wire x1="19.05" y1="5.461" x2="19.685" y2="6.096" width="0.1524" layer="1"/>
+<contactref element="J2" pad="1"/>
+<wire x1="30.226" y1="10.541" x2="30.226" y2="6.731" width="1.016" layer="1"/>
+<contactref element="TP3" pad="S"/>
+<wire x1="32.385" y1="8.89" x2="32.385" y2="7.112" width="0.1524" layer="1"/>
+<wire x1="32.385" y1="7.112" x2="32.004" y2="6.731" width="0.1524" layer="1"/>
+<wire x1="32.004" y1="6.731" x2="30.226" y2="6.731" width="0.1524" layer="1"/>
 </signal>
 <signal name="N$2">
@@
 <wire x1="39.088" y1="30.607" x2="39.624" y2="30.607" width="0.254" layer="1"/>
 <wire x1="39.624" y1="30.607" x2="40.64" y2="29.591" width="0.254" layer="1"/>
+<contactref element="TP2" pad="S"/>
+<wire x1="39.751" y1="12.192" x2="39.751" y2="10.287" width="0.1524" layer="1"/>
+<via x="39.751" y="10.287" extent="1-16" drill="0.254"/>
 </signal>
 <signal name="AGND">
@@
 <via x="41.148" y="10.795" extent="1-16" drill="0.254"/>
 <via x="38.354" y="10.795" extent="1-16" drill="0.254"/>
-<via x="38.354" y="8.382" extent="1-16" drill="0.254"/>
-<via x="41.275" y="8.382" extent="1-16" drill="0.254"/>
-<via x="38.354" y="5.588" extent="1-16" drill="0.254"/>
-<via x="38.354" y="3.048" extent="1-16" drill="0.254"/>
-<via x="41.529" y="3.048" extent="1-16" drill="0.254"/>
+<via x="39.37" y="8.128" extent="1-16" drill="0.254"/>
+<via x="41.275" y="8.128" extent="1-16" drill="0.254"/>
+<via x="38.227" y="5.08" extent="1-16" drill="0.254"/>
+<via x="34.29" y="3.175" extent="1-16" drill="0.254"/>
+<via x="39.37" y="3.175" extent="1-16" drill="0.254"/>
 <via x="48.006" y="3.048" extent="1-16" drill="0.254"/>
 <via x="47.879" y="6.096" extent="1-16" drill="0.254"/>
@@
 <via x="13.589" y="13.208" extent="1-16" drill="0.254"/>
 <via x="31.75" y="10.16" extent="1-16" drill="0.254"/>
-<via x="31.75" y="8.001" extent="1-16" drill="0.254"/>
+<via x="31.242" y="8.001" extent="1-16" drill="0.254"/>
 <via x="31.75" y="13.716" extent="1-16" drill="0.254"/>
 <via x="31.75" y="16.51" extent="1-16" drill="0.254"/>
@@
 <via x="8.89" y="5.334" extent="1-16" drill="0.254"/>
 <via x="8.89" y="3.048" extent="1-16" drill="0.254"/>
-<via x="11.684" y="3.048" extent="1-16" drill="0.254"/>
+<via x="12.192" y="3.429" extent="1-16" drill="0.254"/>
 <via x="11.684" y="5.334" extent="1-16" drill="0.254"/>
-<via x="14.351" y="3.048" extent="1-16" drill="0.254"/>
+<via x="14.478" y="3.429" extent="1-16" drill="0.254"/>
 <via x="17.018" y="3.048" extent="1-16" drill="0.254"/>
 <via x="26.67" y="3.175" extent="1-16" drill="0.254"/>
@@
 <via x="31.75" y="5.461" extent="1-16" drill="0.254"/>
 <via x="28.829" y="13.716" extent="1-16" drill="0.254"/>
-<via x="34.29" y="3.048" extent="1-16" drill="0.254"/>
+<via x="31.623" y="3.175" extent="1-16" drill="0.254"/>
 <via x="1.27" y="10.414" extent="1-16" drill="0.254"/>
 <via x="3.81" y="10.541" extent="1-16" drill="0.254"/>
+<contactref element="TP1" pad="G"/>
+<contactref element="TP3" pad="G"/>
+<contactref element="TP2" pad="G"/>
+<via x="36.83" y="3.175" extent="1-16" drill="0.254"/>
+<via x="41.91" y="3.175" extent="1-16" drill="0.254"/>
+<via x="34.29" y="8.763" extent="1-16" drill="0.254"/>
+<via x="34.29" y="6.223" extent="1-16" drill="0.254"/>
+<via x="34.29" y="13.843" extent="1-16" drill="0.254"/>
+<via x="44.196" y="8.128" extent="1-16" drill="0.254"/>
+<via x="60.833" y="8.128" extent="1-16" drill="0.254"/>
+<via x="57.912" y="8.128" extent="1-16" drill="0.254"/>
+<via x="55.245" y="8.128" extent="1-16" drill="0.254"/>
+<via x="50.038" y="8.128" extent="1-16" drill="0.254"/>
+<via x="46.99" y="8.128" extent="1-16" drill="0.254"/>
 </signal>
 <signal name="N$4">
@@
 <wire x1="9.017" y1="8.412" x2="9.017" y2="9.398" width="0.254" layer="1"/>
 <wire x1="9.017" y1="8.412" x2="7.396" y2="8.412" width="0.4064" layer="1"/>
+<contactref element="TP1" pad="S"/>
+<wire x1="9.017" y1="7.112" x2="9.017" y2="9.398" width="0.1524" layer="16"/>
+<wire x1="7.747" y1="3.429" x2="7.747" y2="4.826" width="0.1524" layer="1"/>
+<via x="7.747" y="4.826" extent="1-16" drill="0.254"/>
+<wire x1="7.747" y1="4.826" x2="7.747" y2="5.842" width="0.1524" layer="16"/>
+<wire x1="7.747" y1="5.842" x2="9.017" y2="7.112" width="0.1524" layer="16"/>
 </signal>
 <signal name="N$7">
@@
 <via x="54.737" y="18.034" extent="1-16" drill="0.254"/>
 <wire x1="54.737" y1="18.034" x2="52.451" y2="18.034" width="0.1524" layer="16"/>
-<wire x1="52.451" y1="18.034" x2="51.308" y2="16.891" width="0.1524" layer="16"/>
-<wire x1="51.308" y1="16.891" x2="45.593" y2="16.891" width="0.1524" layer="16"/>
-<wire x1="45.593" y1="16.891" x2="42.164" y2="20.447" width="0.1524" layer="16"/>
+<wire x1="52.451" y1="18.034" x2="51.435" y2="17.018" width="0.1524" layer="16"/>
+<wire x1="51.435" y1="17.018" x2="45.466" y2="17.018" width="0.1524" layer="16"/>
+<wire x1="45.466" y1="17.018" x2="42.164" y2="20.447" width="0.1524" layer="16"/>
 <wire x1="42.164" y1="20.447" x2="42.037" y2="25.273" width="0.1524" layer="16"/>
 <wire x1="42.037" y1="25.273" x2="41.783" y2="25.527" width="0.1524" layer="16"/>

Commit message: Small stitching tweaks.  Last tweaks, I promise!
Routing:
- net AGND: vias 400 -> 402
Changed lines of the file:
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@@
 </element>
 <element name="R4" library="passives" package="R0603" value="330" x="26.797" y="16.002" smashed="yes">
-<attribute name="NAME" x="28.575" y="15.367" size="1.27" layer="25" font="vector"/>
+<attribute name="NAME" x="28.575" y="15.621" size="1.27" layer="25" font="vector"/>
 <attribute name="PN" value="RC0603FR-07330RL" x="26.797" y="16.002" size="1.778" layer="27" display="off"/>
 </element>
@@
 </element>
 <element name="X1" library="crystals" package="EPSON-TSX-3225" value="26MHz" x="42.672" y="18.669" smashed="yes">
-<attribute name="NAME" x="40.386" y="15.24" size="1.27" layer="25" font="vector"/>
+<attribute name="NAME" x="40.259" y="15.24" size="1.27" layer="25" font="vector"/>
 <attribute name="PN" value="TSX-3225 26.0000MF09Z-AC3" x="42.672" y="18.669" size="1.778" layer="27" display="off"/>
 </element>
@@
 </element>
 <element name="C7" library="passives" package="C0402" value="14pF" x="39.37" y="18.669" smashed="yes" rot="R270">
-<attribute name="NAME" x="38.735" y="17.399" size="1.27" layer="25" font="vector" rot="R270"/>
+<attribute name="NAME" x="38.735" y="17.526" size="1.27" layer="25" font="vector" rot="R270"/>
 <attribute name="PN" value="GJM1555C1H140GB01D" x="39.37" y="18.669" size="1.778" layer="27" rot="R270" display="off"/>
 </element>
@@
 <element name="R16" library="passives" package="R0603" value="330" x="26.797" y="17.78" smashed="yes">
 <attribute name="PN" value="RC0603FR-07330RL" x="26.797" y="17.78" size="1.778" layer="27" display="off"/>
-<attribute name="NAME" x="28.575" y="17.145" size="1.27" layer="25" font="vector"/>
+<attribute name="NAME" x="28.575" y="17.272" size="1.27" layer="25" font="vector"/>
 <attribute name="VALUE" x="25.019" y="19.05" size="1.27" layer="27"/>
 </element>
@@
 <via x="63.5" y="27.051" extent="1-16" drill="0.254"/>
 <via x="63.5" y="24.638" extent="1-16" drill="0.254"/>
-<via x="63.373" y="19.685" extent="1-16" drill="0.254"/>
-<via x="63.5" y="13.716" extent="1-16" drill="0.254"/>
-<via x="63.5" y="10.668" extent="1-16" drill="0.254"/>
-<via x="63.5" y="8.128" extent="1-16" drill="0.254"/>
+<via x="62.992" y="19.431" extent="1-16" drill="0.254"/>
+<via x="62.992" y="13.716" extent="1-16" drill="0.254"/>
+<via x="63.119" y="10.668" extent="1-16" drill="0.254"/>
+<via x="63.119" y="8.128" extent="1-16" drill="0.254"/>
 <via x="63.5" y="5.588" extent="1-16" drill="0.254"/>
 <via x="63.5" y="3.048" extent="1-16" drill="0.254"/>
-<via x="60.833" y="10.668" extent="1-16" drill="0.254"/>
-<via x="57.912" y="10.668" extent="1-16" drill="0.254"/>
-<via x="53.975" y="10.795" extent="1-16" drill="0.254"/>
+<via x="59.944" y="10.668" extent="1-16" drill="0.254"/>
+<via x="56.642" y="10.668" extent="1-16" drill="0.254"/>
+<via x="53.213" y="10.795" extent="1-16" drill="0.254"/>
 <via x="50.038" y="10.795" extent="1-16" drill="0.254"/>
 <via x="46.99" y="10.795" extent="1-16" drill="0.254"/>
-<via x="44.196" y="10.795" extent="1-16" drill="0.254"/>
-<via x="41.148" y="10.795" extent="1-16" drill="0.254"/>
+<via x="43.942" y="10.795" extent="1-16" drill="0.254"/>
+<via x="40.64" y="10.795" extent="1-16" drill="0.254"/>
 <via x="38.354" y="10.795" extent="1-16" drill="0.254"/>
 <via x="39.37" y="8.128" extent="1-16" drill="0.254"/>
@@
 <via x="57.658" y="3.429" extent="1-16" drill="0.254"/>
 <via x="57.658" y="6.096" extent="1-16" drill="0.254"/>
-<via x="52.578" y="8.89" extent="1-16" drill="0.254"/>
-<via x="53.848" y="13.716" extent="1-16" drill="0.254"/>
+<via x="53.213" y="8.128" extent="1-16" drill="0.254"/>
+<via x="53.213" y="13.716" extent="1-16" drill="0.254"/>
 <via x="50.038" y="13.716" extent="1-16" drill="0.254"/>
-<via x="46.863" y="13.589" extent="1-16" drill="0.254"/>
-<via x="44.069" y="13.589" extent="1-16" drill="0.254"/>
-<via x="41.148" y="13.589" extent="1-16" drill="0.254"/>
+<via x="46.863" y="13.716" extent="1-16" drill="0.254"/>
+<via x="43.815" y="13.716" extent="1-16" drill="0.254"/>
+<via x="40.64" y="13.716" extent="1-16" drill="0.254"/>
 <via x="37.338" y="13.843" extent="1-16" drill="0.254"/>
 <via x="46.863" y="16.51" extent="1-16" drill="0.254"/>
-<via x="43.942" y="16.256" extent="1-16" drill="0.254"/>
-<via x="46.736" y="18.034" extent="1-16" drill="0.254"/>
+<via x="43.815" y="16.51" extent="1-16" drill="0.254"/>
+<via x="46.863" y="18.034" extent="1-16" drill="0.254"/>
 <via x="39.37" y="20.066" extent="1-16" drill="0.254"/>
 <via x="49.911" y="16.51" extent="1-16" drill="0.254"/>
-<via x="49.657" y="19.558" extent="1-16" drill="0.254"/>
+<via x="49.53" y="19.431" extent="1-16" drill="0.254"/>
 <via x="46.863" y="21.717" extent="1-16" drill="0.254"/>
-<via x="57.785" y="13.716" extent="1-16" drill="0.254"/>
-<via x="60.706" y="13.716" extent="1-16" drill="0.254"/>
-<via x="57.785" y="19.685" extent="1-16" drill="0.254"/>
+<via x="56.642" y="13.716" extent="1-16" drill="0.254"/>
+<via x="59.944" y="13.716" extent="1-16" drill="0.254"/>
+<via x="56.642" y="19.431" extent="1-16" drill="0.254"/>
 <via x="57.785" y="16.764" extent="1-16" drill="0.254"/>
-<via x="54.61" y="19.685" extent="1-16" drill="0.254"/>
-<via x="60.579" y="19.685" extent="1-16" drill="0.254"/>
+<via x="53.594" y="19.431" extent="1-16" drill="0.254"/>
+<via x="59.944" y="19.431" extent="1-16" drill="0.254"/>
 <via x="59.817" y="16.764" extent="1-16" drill="0.254"/>
 <via x="59.817" y="31.242" extent="1-16" drill="0.254"/>
@@
 <via x="11.303" y="20.574" extent="1-16" drill="0.254"/>
 <via x="13.589" y="20.574" extent="1-16" drill="0.254"/>
-<via x="13.589" y="18.288" extent="1-16" drill="0.254"/>
+<via x="13.97" y="18.288" extent="1-16" drill="0.254"/>
 <via x="11.303" y="18.288" extent="1-16" drill="0.254"/>
-<via x="13.589" y="15.748" extent="1-16" drill="0.254"/>
+<via x="13.97" y="15.748" extent="1-16" drill="0.254"/>
 <via x="11.303" y="15.748" extent="1-16" drill="0.254"/>
 <via x="16.891" y="18.415" extent="1-16" drill="0.254"/>
@@
 <via x="16.891" y="20.574" extent="1-16" drill="0.254"/>
 <via x="16.891" y="13.208" extent="1-16" drill="0.254"/>
-<via x="13.589" y="13.208" extent="1-16" drill="0.254"/>
+<via x="13.97" y="13.208" extent="1-16" drill="0.254"/>
 <via x="31.75" y="10.16" extent="1-16" drill="0.254"/>
 <via x="31.242" y="8.001" extent="1-16" drill="0.254"/>
@@
 <via x="34.544" y="18.923" extent="1-16" drill="0.254"/>
 <via x="31.75" y="18.923" extent="1-16" drill="0.254"/>
-<via x="34.671" y="21.209" extent="1-16" drill="0.254"/>
+<via x="34.544" y="21.209" extent="1-16" drill="0.254"/>
 <via x="28.956" y="18.923" extent="1-16" drill="0.254"/>
 <via x="25.908" y="18.923" extent="1-16" drill="0.254"/>
@@
 <via x="26.416" y="12.7" extent="1-16" drill="0.254"/>
 <via x="31.75" y="5.461" extent="1-16" drill="0.254"/>
-<via x="28.829" y="13.716" extent="1-16" drill="0.254"/>
+<via x="28.956" y="13.716" extent="1-16" drill="0.254"/>
 <via x="31.623" y="3.175" extent="1-16" drill="0.254"/>
 <via x="1.27" y="10.414" extent="1-16" drill="0.254"/>
@@
 <via x="34.29" y="13.843" extent="1-16" drill="0.254"/>
 <via x="44.196" y="8.128" extent="1-16" drill="0.254"/>
-<via x="60.833" y="8.128" extent="1-16" drill="0.254"/>
-<via x="57.912" y="8.128" extent="1-16" drill="0.254"/>
-<via x="55.245" y="8.128" extent="1-16" drill="0.254"/>
+<via x="60.071" y="8.128" extent="1-16" drill="0.254"/>
+<via x="56.642" y="8.128" extent="1-16" drill="0.254"/>
 <via x="50.038" y="8.128" extent="1-16" drill="0.254"/>
 <via x="46.99" y="8.128" extent="1-16" drill="0.254"/>
+<via x="40.64" y="16.51" extent="1-16" drill="0.254"/>
+<via x="28.956" y="16.51" extent="1-16" drill="0.254"/>
+<via x="11.557" y="13.208" extent="1-16" drill="0.254"/>
 </signal>
 <signal name="N$4">
