File: projects/cec-wifi-bridge-rev-a/cec-wifi-bridge-rev-a.brd (EAGLE design)
At the start: 75.9 x 36.1 mm, 59 parts, among them J1 DX4R005HJ5R2000, J3 DEBUG, J4 10029449-001RLF, J5 PROGRAM, T1 MMBT3904, T2 MMBT3904, U1 MCP73831/2/OT, U2 TPS61200DRC, U3 ESP8266EX, U4 SPI-FLASH-SOIC8, X1 26MHz

Commit message: Final layout tweaks before locking rev A.
We've given the TPS61200 its own power ground, hopefully quashing as
much noise as possible off the main ground, keeping RF performance high.

I lied, and went back to adjust the stitching.  We should have our
stitching on a 100 mil grid consistently, with a few exceptions to deal
with component placement.

Also fixed a bug where we had a decoupling cap on a configuration pin
instead of a supply pin.
Parts:
- moved C10 9.92 mm to (45.8, 22.7), turned to 0 degrees
- moved U$2 2.04 mm to (49.5, 19.6)
- moved C5 1.45 mm to (26.4, 8.38), turned to 270 degrees
- moved C7 1.28 mm to (39.2, 17.4), turned to 0 degrees
- moved C6 1.17 mm to (46.1, 19.8), turned to 0 degrees
- moved R12 1.05 mm to (25.3, 22.7)
- moved R3 0.90 mm to (20.4, 3.17), turned to 0 degrees
- moved R2 0.72 mm to (20.4, 4.32), turned to 180 degrees
- moved C2 0.68 mm to (22.5, 3.17), turned to 0 degrees
- moved L1 0.65 mm to (20.4, 10.9)
- moved J5 0.63 mm to (35.7, 9.40)
- moved C4 0.52 mm to (24.6, 8.13), turned to 270 degrees
- moved D3 0.51 mm to (23.1, 17.3)
- moved R16 0.51 mm to (26.8, 17.3)
- moved D1 0.51 mm to (23.1, 15.5)
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Routing:
- net VBAT: track 37.5 -> 20.0 mm
- net TCK: track 30.8 -> 18.7 mm, vias 2 -> 1
- net !RST: track 47.1 -> 53.5 mm
- net TDI: track 18.3 -> 12.9 mm
- net TDO: track 17.4 -> 21.7 mm
- net +3V3: track 41.9 -> 39.7 mm
- net UART_TX: track 16.4 -> 17.7 mm
- net N$25: track 15.7 -> 14.9 mm
- net CEC_TX: track 18.3 -> 17.5 mm
- net N$7: track 24.1 -> 23.4 mm
- net CEC_RX: track 22.8 -> 22.2 mm
- net N$22: track 18.4 -> 17.8 mm
- net AGND: vias 402 -> 454
- added copper zone on layer 1, net +3V3

Commit message: A few fixes after testing the rev A1 boards.
Just fixing up a fix issues I found while build/testing the rev A1
boards, namely:
- using wrong footprint for T1/T2
- LEDs way too bright; adjusted series resistors
- used wrong part number for boost converter (ooof!)
- shoved HDMI connector closer to the edge
- added outlines to the various sections
- shuffled around test points and labels
Parts:
- removed TP3: TESTPOINT-WITH-GND, test:TESTPOINT-1.5-WITH-GND
- R16: value 330 -> 270
- R4: value 330 -> 680
- T1, T2: device transistors:SC-70 -> transistors:SOT-23
- U2: value TPS61200DRC -> TPS61201DRC
- moved TP2 9.40 mm to (31.8, 10.7), turned to 90 degrees
- moved U$1 2.54 mm to (14.0, 32.3)
- moved R10 1.27 mm to (19.8, 26.9)
- moved R11 1.27 mm to (19.8, 28.2)
- moved J2 1.17 mm to (30.5, 4.32), turned to 0 degrees
- moved TP1 0.80 mm to (9.27, 4.19)
- moved T1 0.38 mm to (20.6, 21.8), turned to 270 degrees
- moved T2 0.28 mm to (16.9, 27.1), turned to 90 degrees
- moved J4 0.25 mm to (3.68, 25.1)
Connections:
- net AGND: no longer TP3.G
- net VBAT: no longer TP3.S
Routing:
- net VBAT: track 20.0 -> 17.4 mm
- net N$3: track 10.8 -> 8.90 mm
- net N$27: track 3.26 -> 1.52 mm
- net VBUS: track 31.2 -> 30.4 mm
- net HDMI_CEC: track 18.7 -> 19.4 mm
- net +3V3: track 39.7 -> 39.1 mm
- net AGND: vias 454 -> 451
Other:
- board text added: "CEC"
- board text added: "MCU"
- board text added: "PWR"
