File: projects/cec-wifi-bridge-rev-a/cec-wifi-bridge-rev-a.sch (EAGLE design)
At the start: 15 parts, among them J1 DX4R005H91R1500, U1 MCP73831/2/OT, U2 TPS61200DRC

Commit message: Starting to add in the main bits.
Parts:
- added C6, C7: 14pF, passives:CAPACITOR-0402
- added U3: ESP8266EX, espressif:ESP8266EX
- added X1: 26MHz, crystals:GROUNDED-CRYSTAL-EPSON-TSX-3225
Connections:
- new net N$11: C6.1, U3.XTAL_IN, X1.2
- new net N$12: C7.2, U3.XTAL_OUT, X1.1
- net AGND: now also C6.2, C7.1, U3.GND, X1.GND
Changed lines of the file:
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@@
 <part name="J2" library="pin-headers" deviceset="PINHD-1X2" device=""/>
 <part name="SHEET2" library="frames" deviceset="A4L-NODOC" device=""/>
+<part name="U3" library="espressif" deviceset="ESP8266EX" device=""/>
+<part name="X1" library="crystals" deviceset="GROUNDED-CRYSTAL" device="-EPSON-TSX-3225" value="26MHz"/>
+<part name="C6" library="passives" deviceset="CAPACITOR" device="-0402" value="14pF"/>
+<part name="C7" library="passives" deviceset="CAPACITOR" device="-0402" value="14pF"/>
+<part name="AGND13" library="supplies" deviceset="AGND" device=""/>
+<part name="AGND14" library="supplies" deviceset="AGND" device=""/>
 </parts>
 <sheets>
@@
 <instances>
 <instance part="SHEET2" gate="G$1" x="0" y="0"/>
+<instance part="U3" gate="G$1" x="86.36" y="116.84"/>
+<instance part="X1" gate="G$1" x="152.4" y="114.3"/>
+<instance part="C6" gate="G$1" x="160.02" y="109.22"/>
+<instance part="C7" gate="G$1" x="144.78" y="106.68" rot="R180"/>
+<instance part="AGND13" gate="VR1" x="152.4" y="97.79"/>
+<instance part="AGND14" gate="VR1" x="78.74" y="54.61"/>
 </instances>
 <busses>
 </busses>
 <nets>
+<net name="AGND" class="0">
+<segment>
+<pinref part="C7" gate="G$1" pin="1"/>
+<wire x1="144.78" y1="104.14" x2="144.78" y2="102.87" width="0.1524" layer="91"/>
+<pinref part="C6" gate="G$1" pin="2"/>
+<wire x1="144.78" y1="102.87" x2="152.4" y2="102.87" width="0.1524" layer="91"/>
+<wire x1="152.4" y1="102.87" x2="160.02" y2="102.87" width="0.1524" layer="91"/>
+<wire x1="160.02" y1="102.87" x2="160.02" y2="104.14" width="0.1524" layer="91"/>
+<pinref part="AGND13" gate="VR1" pin="AGND"/>
+<wire x1="152.4" y1="100.33" x2="152.4" y2="102.87" width="0.1524" layer="91"/>
+<junction x="152.4" y="102.87"/>
+<pinref part="X1" gate="G$1" pin="GND"/>
+<wire x1="152.4" y1="111.76" x2="152.4" y2="102.87" width="0.1524" layer="91"/>
+</segment>
+<segment>
+<pinref part="U3" gate="G$1" pin="GND"/>
+<pinref part="AGND14" gate="VR1" pin="AGND"/>
+<wire x1="83.82" y1="63.5" x2="78.74" y2="63.5" width="0.1524" layer="91"/>
+<wire x1="78.74" y1="63.5" x2="78.74" y2="57.15" width="0.1524" layer="91"/>
+</segment>
+</net>
+<net name="N$11" class="0">
+<segment>
+<pinref part="U3" gate="G$1" pin="XTAL_IN"/>
+<wire x1="120.65" y1="114.3" x2="130.81" y2="114.3" width="0.1524" layer="91"/>
+<wire x1="130.81" y1="114.3" x2="130.81" y2="123.19" width="0.1524" layer="91"/>
+<wire x1="130.81" y1="123.19" x2="160.02" y2="123.19" width="0.1524" layer="91"/>
+<wire x1="160.02" y1="123.19" x2="160.02" y2="114.3" width="0.1524" layer="91"/>
+<pinref part="X1" gate="G$1" pin="2"/>
+<wire x1="160.02" y1="114.3" x2="154.94" y2="114.3" width="0.1524" layer="91"/>
+<pinref part="C6" gate="G$1" pin="1"/>
+<wire x1="160.02" y1="111.76" x2="160.02" y2="114.3" width="0.1524" layer="91"/>
+<junction x="160.02" y="114.3"/>
+</segment>
+</net>
+<net name="N$12" class="0">
+<segment>
+<pinref part="U3" gate="G$1" pin="XTAL_OUT"/>
+<wire x1="120.65" y1="111.76" x2="133.35" y2="111.76" width="0.1524" layer="91"/>
+<wire x1="133.35" y1="111.76" x2="133.35" y2="114.3" width="0.1524" layer="91"/>
+<pinref part="X1" gate="G$1" pin="1"/>
+<wire x1="133.35" y1="114.3" x2="144.78" y2="114.3" width="0.1524" layer="91"/>
+<pinref part="C7" gate="G$1" pin="2"/>
+<wire x1="144.78" y1="114.3" x2="149.86" y2="114.3" width="0.1524" layer="91"/>
+<wire x1="144.78" y1="111.76" x2="144.78" y2="114.3" width="0.1524" layer="91"/>
+<junction x="144.78" y="114.3"/>
+</segment>
+</net>
 </nets>
 </sheet>

Commit message: Start wiring up the ESP8266.
Parts:
- added J3: DEBUG, pin-headers:PINHD-2X4
- added J4: PROGRAM, pin-headers:PINHD-1X3
- added R5: 12K, passives:RESISTOR-HORIZONTAL-0402
- added R6, R7: 10K, passives:RESISTOR-0402
- added S1: RESET, switches:MOMENTARY-ALPS-SKQG
- added S2: UPLOAD, switches:MOMENTARY-ALPS-SKQG
- added U4: SPI-FLASH-SOIC8, flash:SPI-FLASH-SOIC8
- R1: value 20K -> 2K
Connections:
- new net !RST: J3.1, R7.1, S1.P$2, U3.EXT_RSTB, U3.XPD_DCDC
- new net FLASH_BOOT: R6.1, S2.P$1, U3.GPIO0
- new net N$10: R5.2, U3.RES12K
- new net N$13: J4.1, U3.U0RXD
- new net N$14: J4.2, U3.U0TXD
- new net N$16: J3.2, U3.MTDO
- new net N$17: J3.4, U3.MTCK
- new net N$18: J3.6, U3.MTDI
- new net N$19: J3.8, U3.MTMS
- new net N$20: U3.SD_CLK, U4.SCK
- new net N$21: U3.SD_CMD, U4.!CE
- new net N$22: U3.SD_DATA_1, U4.SI
- new net N$23: U4.SO
- new net N$24: U3.SD_DATA_3, U4.!WP
- new net N$25: U3.SD_DATA_2, U4.!HOLD
- net +3V3: now also R6.2, R7.2, U3.CHIP_EN, U3.GPIO2, U3.VDD3P3, U3.VDDA, U3.VDDD, U3.VDDPST, U3.VDD_RTC, U4.VCC
- net AGND: now also J3.5, J3.7, R5.1, S1.P$1, S2.P$2, U4.GND
Other:
- moved on the sheet: C6, C7, X1

Commit message: Lots of tweaks and changes.
Parts:
- removed J4: PROGRAM, pin-headers:PINHD-1X3
- added ANT1: INVERTED_F_ANTENNA+0, antenna:INVERTED_F_ANTENNA+0
- added C10, C11, C12, C13, C14, C15, C16, C9: 0.1uF, passives:CAPACITOR-0402
- added C8: 5.6pF, passives:CAPACITOR-HORIZONTAL-0402
- added J5: PROGRAM, pin-headers:PINHD-1X5
- R4: value 820 -> 330
Connections:
- net N$17 renamed TCK
- net N$3 renamed VBUS
- removed net N$13: J4.1, U3.U0RXD
- removed net N$14: J4.2, U3.U0TXD
- removed net N$16: J3.2, U3.MTDO
- removed net N$18: J3.6, U3.MTDI
- removed net N$19: J3.8, U3.MTMS
- new net ANT: C8.1, U3.LNA
- new net CEC_IN: U3.GPIO4
- new net CEC_OUT: U3.GPIO5
- new net N$26: ANT1.FEED, C8.2
- new net TDI: J3.8, U3.MTDI
- new net TDO: J3.6, U3.MTDO
- new net TMS: J3.2, U3.MTMS
- new net UART_RX: J5.1, U3.U0RXD
- new net UART_TX: J5.2, U3.U0TXD
- net +3V3: now also C10.1, C11.1, C12.1, C13.1, C14.1, C15.1, C16.1, C9.1; no longer U3.VDD_RTC
- net AGND: now also ANT1.GND, C10.2, C11.2, C12.2, C13.2, C14.2, C15.2, C16.2, C9.2, J5.5
Other:
- note added: "Connectors"
- note added: "Externally, we take in USB power and an HDMI connection and that's the extent of what we need from the outside world. Internally, we have pin headers from programming and debugging. Technically, the ESP8266 doesn't support JTAG debugging yet, but it has pins named as such, so we've broken them out here to be ready for future revs. We also have the antenna on here, but it's not a connector. Just a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"

Commit message: Lots of board layout work.
The board is basically done.

It has a real shape now, things are laid out.  We have fiducials,
alignment holes, rounded edges, the PCB antenna with the proper
setbacks, ground plane stitching, we have our logo in place (!), and
things are generally buttoned up.

We still need to fill out the BOM entirely, as well as clean up the
schematic sheets and add proper titles/descriptions, etc.

Also need to look into bitmap art for open source hardware to start
throwing on the board.  Should probably add the license / attribution
stuff, as well.
Parts:
- added C17: 27pF, passives:CAPACITOR-0402
- added C18: 0.1uF, passives:CAPACITOR-0402
- added D2: 1N4148, diodes:DIODE-SOD123
- added J4: 10029449-001RLF, amphenol:10029449-001RLF
- added R10: 47K, passives:RESISTOR-0402
- added R11, R8: 220, passives:RESISTOR-0402
- added R12: 100K, passives:RESISTOR-0402
- added R13: 27K, passives:RESISTOR-HORIZONTAL-0402
- added R14: 1M, passives:RESISTOR-HORIZONTAL-0402
- added R15: 47K, passives:RESISTOR-HORIZONTAL-0402
- added R9: 470K, passives:RESISTOR-0402
- added T1, T2: MMBT3904, transistors:BJT-NPN-SC-70
- added U$1, U$2, U$3: FIDUCIAL-1MM, fiducials:FIDUCIAL-1MM
Connections:
- removed net CEC_IN: U3.GPIO4
- removed net CEC_OUT: U3.GPIO5
- removed net N$5: R3.1
- new net CEC_RX: R12.1, T1.C, U3.GPIO5
- new net CEC_TX: R15.1, U3.GPIO4
- new net HDMI_CEC: C17.1, D2.C, J4.CEC, R14.2, T2.C
- new net N$15: R8.2, T1.E
- new net N$16: R14.1, R9.2, T1.B
- new net N$18: D2.A, R13.2
- new net N$27: R11.2, T2.E
- new net N$3: C17.2, R10.2, R15.2, T2.B
- net +3V3: now also C18.1, R12.2, R13.1
- net AGND: now also C18.2, J4.GROUND, R10.1, R11.1, R3.1, R8.1, R9.1

Commit message: cleanup
Parts:
- ANT1, J2: BOM (none) -> EXCLUDE
Connections:
- net N$23: now also U3.SD_DATA_0
Other:
- note added: "CEC Interface / Demux"
- note added: "CEC is a one-wire bidirectional protocol, so this circuit allows us to break out the TX and RX into separate lines to allow for an easy software-based implementation."
- note added: "We're using the ESP8266 here to provide simple and effective WiFI control."
- note added: "WiFi / CEC Control"
- moved on the sheet: C17, C6, C7, D2, R10, R11, R12, R13, R14, R15, R5, R6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

Commit message: Filled in BOM and super stitched.
Filled in all of the BOM values.  Also stitches the hell out of the
board.  Realllly stitched it.  Probably overstitched it.
Parts:
- C1: PN (none) -> GRM188R61A475KE15D
- C17: PN (none) -> GRM1555C1H270GA01D
- C2, C4: PN (none) -> GRM155R71H104KE14D
- C3: PN (none) -> GRM21BR61A106KE19L
- C5: PN (none) -> GRM21BR61A226ME51L
- C6, C7: PN (none) -> GJM1555C1H140GB01D
- C8: PN (none) -> GJM1555C1H5R6WB01D
- J1: PN (none) -> DX4R005H91R1500
- J3: PN (none) -> M20-9760446
- J5: PN (none) -> M20-9990546
- R1: PN (none) -> RC0402FR-072KL
- R10, R15: PN (none) -> RC0402FR-0747KL
- R11, R8: PN (none) -> RC0402FR-07220RL
- R12: PN (none) -> RC0402FR-07100KL
- R13: PN (none) -> RC0402FR-0727KL
- R14: PN (none) -> RC0402FR-071ML
- R2: PN (none) -> RC0402FR-072ML
- R3: value 198K -> 196K; PN (none) -> RC0402FR-07196KL
- R4: PN (none) -> RC0805FR-07330RL
- R5: PN (none) -> RC0402FR-0712KL
- R6, R7: PN (none) -> RC0402FR-0710KL
- R9: PN (none) -> RC0402FR-07470KL
- S1, S2: PN (none) -> SKQGAKE010
- T1, T2: PN MMBT3904WT1G -> MMBT3904LT1G
- U1: PN (none) -> MCP73831T-2ACI/OT
- U2: PN (none) -> TPS61200DRCR
- U4: PN (none) -> S25FL116K0XMFI041
- X1: PN (none) -> TSX-3225 26.0000MF09Z-AC3

Commit message: Add BOM parts and adjust alignment holes.
Added the remaining two BOM values.

Adjusted the location of the alignment pin holes so that we can cleanly
fit the LiPo battery on the underside of the board without it being
under the PCB antenna and without it being too close to the HDMI
through-hole pins.
Parts:
- L1: PN (none) -> XPL2010-222MLB
Changed lines of the file:
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@@
 </part>
 <part name="AGND12" library="supplies" deviceset="AGND" device=""/>
-<part name="L1" library="passives" deviceset="INDUCTOR-HORIZONTAL" device="-XPL2010" value="2.2uH"/>
+<part name="L1" library="passives" deviceset="INDUCTOR-HORIZONTAL" device="-XPL2010" value="2.2uH">
+<attribute name="PN" value="XPL2010-222MLB"/>
+</part>
 <part name="J2" library="pin-headers" deviceset="PINHD-1X2" device="">
 <attribute name="BOM" value="EXCLUDE"/>
@@
 </instance>
 <instance part="AGND12" gate="VR1" x="121.92" y="68.58"/>
-<instance part="L1" gate="G$1" x="190.5" y="118.11"/>
+<instance part="L1" gate="G$1" x="190.5" y="118.11">
+<attribute name="PN" x="190.5" y="118.11" size="1.778" layer="96" display="off"/>
+</instance>
 <instance part="J2" gate="G$1" x="144.78" y="110.49">
 <attribute name="BOM" x="144.78" y="110.49" size="5.08" layer="96" display="off"/>

Commit message: Add LED and more board tweaking.
Added another LED after realizing that STAT on the battery charger IC is
actually tri-state -- thanks, Adafruit!  This means we can now show when
the battery is charging and when it's full, wee!

Also moved bits and pieces around on the board.  Spread out the
stitching vias, moved vias out of the way of the silkscreen, etc etc.
Parts:
- added D3: 3.2V, 5mA, dialight:DIALIGHT-598-MICROSMD-0603
- added R16: 330, passives:RESISTOR-HORIZONTAL-0603
- D1: value 2V, 4mA -> 2V, 5mA
- R4: device passives:RESISTOR-HORIZONTAL-0805 -> passives:RESISTOR-HORIZONTAL-0603; PN RC0805FR-07330RL -> RC0603FR-07330RL
Connections:
- new net N$5: D3.A, R16.1
- net AGND: now also D3.C
- net N$7: now also R16.2
Other:
- moved on the sheet: C1, R1, U1
Changed lines of the file:
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@@
 <setting verticaltext="up"/>
 </settings>
-<grid distance="0.1" unitdist="inch" unit="inch" style="lines" multiple="1" display="no" altdistance="0.01" altunitdist="inch" altunit="inch"/>
+<grid distance="0.05" unitdist="inch" unit="inch" style="lines" multiple="1" display="no" altdistance="0.01" altunitdist="inch" altunit="inch"/>
 <layers>
 <layer number="1" name="Top" color="4" fill="1" visible="no" active="no"/>
@@
 <part name="AGND9" library="supplies" deviceset="AGND" device=""/>
 <part name="AGND10" library="supplies" deviceset="AGND" device=""/>
-<part name="D1" library="dialight" deviceset="DIALIGHT-598-MICROSMD" device="-0603" value="2V, 4mA">
+<part name="D1" library="dialight" deviceset="DIALIGHT-598-MICROSMD" device="-0603" value="2V, 5mA">
 <attribute name="PN" value="598-8020-107F"/>
 </part>
-<part name="R4" library="passives" deviceset="RESISTOR-HORIZONTAL" device="-0805" value="330">
-<attribute name="PN" value="RC0805FR-07330RL"/>
+<part name="R4" library="passives" deviceset="RESISTOR-HORIZONTAL" device="-0603" value="330">
+<attribute name="PN" value="RC0603FR-07330RL"/>
 </part>
 <part name="AGND11" library="supplies" deviceset="AGND" device=""/>
@@
 <attribute name="BOM" value="EXCLUDE"/>
 </part>
+<part name="R16" library="passives" deviceset="RESISTOR-HORIZONTAL" device="-0603" value="330">
+<attribute name="PN" value="RC0603FR-07330RL"/>
+</part>
+<part name="D3" library="dialight" deviceset="DIALIGHT-598-MICROSMD" device="-0603" value="3.2V, 5mA">
+<attribute name="PN" value="598-8081-107F"/>
+</part>
+<part name="AGND27" library="supplies" deviceset="AGND" device=""/>
 </parts>
 <sheets>
@@
 <attribute name="BOM" x="0" y="0" size="5.08" layer="96" display="off"/>
 </instance>
-<instance part="U1" gate="G$1" x="71.12" y="102.87">
-<attribute name="PN" x="71.12" y="102.87" size="1.778" layer="96" display="off"/>
+<instance part="U1" gate="G$1" x="76.2" y="102.87">
+<attribute name="PN" x="76.2" y="102.87" size="1.778" layer="96" display="off"/>
 </instance>
 <instance part="U2" gate="G$1" x="180.34" y="102.87">
 <attribute name="PN" x="180.34" y="102.87" size="1.778" layer="96" display="off"/>
 </instance>
-<instance part="C1" gate="G$1" x="106.68" y="90.17">
-<attribute name="PN" x="106.68" y="90.17" size="1.778" layer="96" display="off"/>
-</instance>
-<instance part="R1" gate="G$1" x="95.25" y="88.9">
-<attribute name="PN" x="95.25" y="88.9" size="1.778" layer="96" display="off"/>
+<instance part="C1" gate="G$1" x="111.76" y="90.17">
+<attribute name="PN" x="111.76" y="90.17" size="1.778" layer="96" display="off"/>
+</instance>
+<instance part="R1" gate="G$1" x="101.6" y="88.9">
+<attribute name="PN" x="101.6" y="88.9" size="1.778" layer="96" display="off"/>
 </instance>
 <instance part="R2" gate="G$1" x="160.02" y="93.98">
@@
 </instance>
 <instance part="+3V1" gate="G$1" x="238.76" y="115.57"/>
-<instance part="AGND1" gate="VR1" x="64.77" y="68.58"/>
+<instance part="AGND1" gate="VR1" x="69.85" y="68.58"/>
 <instance part="AGND2" gate="VR1" x="173.99" y="68.58"/>
 <instance part="AGND3" gate="VR1" x="209.55" y="68.58"/>
 <instance part="AGND4" gate="VR1" x="238.76" y="68.58"/>
 <instance part="AGND5" gate="VR1" x="223.52" y="68.58"/>
-<instance part="AGND6" gate="VR1" x="106.68" y="68.58"/>
-<instance part="AGND7" gate="VR1" x="95.25" y="68.58"/>
+<instance part="AGND6" gate="VR1" x="111.76" y="68.58"/>
+<instance part="AGND7" gate="VR1" x="101.6" y="68.58"/>
 <instance part="AGND8" gate="VR1" x="133.35" y="68.58"/>
 <instance part="AGND9" gate="VR1" x="147.32" y="68.58"/>
@@
 <attribute name="PN" x="58.42" y="97.79" size="1.778" layer="96" display="off"/>
 </instance>
-<instance part="AGND12" gate="VR1" x="121.92" y="68.58"/>
+<instance part="AGND12" gate="VR1" x="124.46" y="68.58"/>
 <instance part="L1" gate="G$1" x="190.5" y="118.11">
 <attribute name="PN" x="190.5" y="118.11" size="1.778" layer="96" display="off"/>
@@
 <attribute name="PN" x="121.92" y="34.29" size="2.54" layer="96" display="off"/>
 </instance>
+<instance part="R16" gate="G$1" x="58.42" y="88.9">
+<attribute name="PN" x="58.42" y="88.9" size="1.778" layer="96" display="off"/>
+</instance>
+<instance part="D3" gate="G$1" x="45.72" y="88.9" rot="R180">
+<attribute name="PN" x="45.72" y="88.9" size="1.778" layer="96" rot="R180" display="off"/>
+</instance>
+<instance part="AGND27" gate="VR1" x="36.83" y="68.58"/>
 </instances>
 <busses>
@@
 <wire x1="175.26" y1="100.33" x2="160.02" y2="100.33" width="0.1524" layer="91"/>
 <wire x1="160.02" y1="100.33" x2="133.35" y2="100.33" width="0.1524" layer="91"/>
-<wire x1="133.35" y1="100.33" x2="106.68" y2="100.33" width="0.1524" layer="91"/>
-<wire x1="106.68" y1="100.33" x2="91.44" y2="100.33" width="0.1524" layer="91"/>
+<wire x1="133.35" y1="100.33" x2="111.76" y2="100.33" width="0.1524" layer="91"/>
+<wire x1="111.76" y1="100.33" x2="96.52" y2="100.33" width="0.1524" layer="91"/>
 <wire x1="177.8" y1="97.79" x2="175.26" y2="97.79" width="0.1524" layer="91"/>
 <wire x1="175.26" y1="97.79" x2="175.26" y2="100.33" width="0.1524" layer="91"/>
@@
 <junction x="133.35" y="100.33"/>
 <pinref part="C1" gate="G$1" pin="1"/>
-<wire x1="106.68" y1="92.71" x2="106.68" y2="100.33" width="0.1524" layer="91"/>
-<junction x="106.68" y="100.33"/>
+<wire x1="111.76" y1="92.71" x2="111.76" y2="100.33" width="0.1524" layer="91"/>
+<junction x="111.76" y="100.33"/>
 <wire x1="142.24" y1="113.03" x2="133.35" y2="113.03" width="0.1524" layer="91"/>
 <wire x1="133.35" y1="113.03" x2="133.35" y2="100.33" width="0.1524" layer="91"/>
@@
 <pinref part="U1" gate="G$1" pin="GND"/>
 <pinref part="AGND1" gate="VR1" pin="AGND"/>
-<wire x1="68.58" y1="92.71" x2="64.77" y2="92.71" width="0.1524" layer="91"/>
-<wire x1="64.77" y1="92.71" x2="64.77" y2="71.12" width="0.1524" layer="91"/>
+<wire x1="73.66" y1="92.71" x2="69.85" y2="92.71" width="0.1524" layer="91"/>
+<wire x1="69.85" y1="92.71" x2="69.85" y2="71.12" width="0.1524" layer="91"/>
 </segment>
 <segment>
 <pinref part="AGND7" gate="VR1" pin="AGND"/>
 <pinref part="R1" gate="G$1" pin="1"/>
-<wire x1="95.25" y1="71.12" x2="95.25" y2="83.82" width="0.1524" layer="91"/>
+<wire x1="101.6" y1="71.12" x2="101.6" y2="83.82" width="0.1524" layer="91"/>
 </segment>
 <segment>
 <pinref part="AGND6" gate="VR1" pin="AGND"/>
 <pinref part="C1" gate="G$1" pin="2"/>
-<wire x1="106.68" y1="71.12" x2="106.68" y2="85.09" width="0.1524" layer="91"/>
+<wire x1="111.76" y1="71.12" x2="111.76" y2="85.09" width="0.1524" layer="91"/>
 </segment>
 <segment>
@@
 </segment>
 <segment>
-<wire x1="142.24" y1="110.49" x2="121.92" y2="110.49" width="0.1524" layer="91"/>
-<wire x1="121.92" y1="110.49" x2="121.92" y2="71.12" width="0.1524" layer="91"/>
+<wire x1="142.24" y1="110.49" x2="124.46" y2="110.49" width="0.1524" layer="91"/>
+<wire x1="124.46" y1="110.49" x2="124.46" y2="71.12" width="0.1524" layer="91"/>
 <pinref part="AGND12" gate="VR1" pin="AGND"/>
 <pinref part="J2" gate="G$1" pin="2"/>
@@
 <pinref part="R3" gate="G$1" pin="1"/>
 </segment>
+<segment>
+<pinref part="D3" gate="G$1" pin="C"/>
+<wire x1="43.18" y1="88.9" x2="36.83" y2="88.9" width="0.1524" layer="91"/>
+<wire x1="36.83" y1="88.9" x2="36.83" y2="71.12" width="0.1524" layer="91"/>
+<pinref part="AGND27" gate="VR1" pin="AGND"/>
+</segment>
 </net>
 <net name="N$4" class="0">
@@
 <pinref part="U1" gate="G$1" pin="PROG"/>
 <pinref part="R1" gate="G$1" pin="2"/>
-<wire x1="91.44" y1="97.79" x2="95.25" y2="97.79" width="0.1524" layer="91"/>
-<wire x1="95.25" y1="97.79" x2="95.25" y2="93.98" width="0.1524" layer="91"/>
+<wire x1="96.52" y1="97.79" x2="101.6" y2="97.79" width="0.1524" layer="91"/>
+<wire x1="101.6" y1="97.79" x2="101.6" y2="93.98" width="0.1524" layer="91"/>
 </segment>
 </net>
@@
 <net name="VBUS" class="0">
 <segment>
-<wire x1="38.1" y1="109.22" x2="63.5" y2="109.22" width="0.1524" layer="91"/>
-<wire x1="63.5" y1="109.22" x2="63.5" y2="100.33" width="0.1524" layer="91"/>
+<wire x1="38.1" y1="109.22" x2="69.85" y2="109.22" width="0.1524" layer="91"/>
+<wire x1="69.85" y1="109.22" x2="69.85" y2="100.33" width="0.1524" layer="91"/>
 <pinref part="U1" gate="G$1" pin="VDD"/>
-<wire x1="63.5" y1="100.33" x2="68.58" y2="100.33" width="0.1524" layer="91"/>
+<wire x1="69.85" y1="100.33" x2="73.66" y2="100.33" width="0.1524" layer="91"/>
 <pinref part="D1" gate="G$1" pin="A"/>
 <wire x1="43.18" y1="97.79" x2="38.1" y2="97.79" width="0.1524" layer="91"/>
@@
 <pinref part="R4" gate="G$1" pin="2"/>
 <pinref part="U1" gate="G$1" pin="STAT"/>
-<wire x1="63.5" y1="97.79" x2="68.58" y2="97.79" width="0.1524" layer="91"/>
+<wire x1="63.5" y1="97.79" x2="66.04" y2="97.79" width="0.1524" layer="91"/>
+<pinref part="R16" gate="G$1" pin="2"/>
+<wire x1="66.04" y1="97.79" x2="73.66" y2="97.79" width="0.1524" layer="91"/>
+<wire x1="63.5" y1="88.9" x2="66.04" y2="88.9" width="0.1524" layer="91"/>
+<wire x1="66.04" y1="88.9" x2="66.04" y2="97.79" width="0.1524" layer="91"/>
+<junction x="66.04" y="97.79"/>
 </segment>
 </net>
@@
 </segment>
 </net>
+<net name="N$5" class="0">
+<segment>
+<pinref part="R16" gate="G$1" pin="1"/>
+<pinref part="D3" gate="G$1" pin="A"/>
+<wire x1="53.34" y1="88.9" x2="50.8" y2="88.9" width="0.1524" layer="91"/>
+</segment>
+</net>
