File: projects/cec-wifi-bridge-rev-a/cec-wifi-bridge-rev-a.sch (EAGLE design)
At the start: 56 parts, among them J1 DX4R005H91R1500, J3 DEBUG, J4 10029449-001RLF, J5 PROGRAM, T1 MMBT3904, T2 MMBT3904, U1 MCP73831/2/OT, U2 TPS61200DRC, U3 ESP8266EX, U4 SPI-FLASH-SOIC8, X1 26MHz

Commit message: Switch to DX4R005HJ5R2000 for USB connector.
The other version we were using had no 3D model available from JAE, so I
found one that did, so we can properly design the enclosure and model it
all assembled.
Parts:
- J1: value DX4R005H91R1500 -> DX4R005HJ5R2000; device jae:DX4R005H91R1500 -> jae:DX4R005HJ5R2000; PN DX4R005H91R1500 -> DX4R005HJ5R2000
Changed lines of the file:
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@@
 <setting verticaltext="up"/>
 </settings>
-<grid distance="0.05" unitdist="inch" unit="inch" style="lines" multiple="1" display="no" altdistance="0.01" altunitdist="inch" altunit="inch"/>
+<grid distance="0.1" unitdist="inch" unit="inch" style="lines" multiple="1" display="no" altdistance="0.01" altunitdist="inch" altunit="inch"/>
 <layers>
 <layer number="1" name="Top" color="4" fill="1" visible="no" active="no"/>
@@
 </part>
 <part name="AGND11" library="supplies" deviceset="AGND" device=""/>
-<part name="J1" library="jae" deviceset="DX4R005H91R1500" device="">
-<attribute name="PN" value="DX4R005H91R1500"/>
+<part name="J1" library="jae" deviceset="DX4R005HJ5R2000" device="">
+<attribute name="PN" value="DX4R005HJ5R2000"/>
 </part>
 <part name="AGND12" library="supplies" deviceset="AGND" device=""/>

Commit message: Add part number for ESP8266.
Parts:
- U3: PN (none) -> ESP8266EX
Changed lines of the file:
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@@
 <attribute name="BOM" value="EXCLUDE"/>
 </part>
-<part name="U3" library="espressif" deviceset="ESP8266EX" device=""/>
+<part name="U3" library="espressif" deviceset="ESP8266EX" device="">
+<attribute name="PN" value="ESP8266EX"/>
+</part>
 <part name="X1" library="crystals" deviceset="GROUNDED-CRYSTAL" device="-EPSON-TSX-3225" value="26MHz">
 <attribute name="PN" value="TSX-3225 26.0000MF09Z-AC3"/>
@@
 <attribute name="BOM" x="0" y="0" size="5.08" layer="96" display="off"/>
 </instance>
-<instance part="U3" gate="G$1" x="86.36" y="99.06"/>
+<instance part="U3" gate="G$1" x="86.36" y="99.06">
+<attribute name="PN" x="86.36" y="99.06" size="1.778" layer="96" display="off"/>
+</instance>
 <instance part="X1" gate="G$1" x="198.12" y="121.92">
 <attribute name="PN" x="198.12" y="121.92" size="1.778" layer="96" display="off"/>

Commit message: Add testpoints for the power rails.
Parts:
- added TP1, TP2, TP3: TESTPOINT-WITH-GND, test:TESTPOINT-WITH-GND
Connections:
- removed net N$1: C1.1, C3.1, J2.1, L1.2, R2.2, U1.VBAT, U2.EN, U2.PS, U2.VIN
- new net VBAT: C1.1, C3.1, J2.1, L1.2, R2.2, TP3.S, U1.VBAT, U2.EN, U2.PS, U2.VIN
- net +3V3: now also TP2.S
- net AGND: now also TP1.G, TP2.G, TP3.G
- net VBUS: now also TP1.S
Other:
- moved on the sheet: ANT1, C8, J1, J3, J4, J5

Commit message: Final layout tweaks before locking rev A.
We've given the TPS61200 its own power ground, hopefully quashing as
much noise as possible off the main ground, keeping RF performance high.

I lied, and went back to adjust the stitching.  We should have our
stitching on a 100 mil grid consistently, with a few exceptions to deal
with component placement.

Also fixed a bug where we had a decoupling cap on a configuration pin
instead of a supply pin.
Parts:
- TP1, TP2, TP3: BOM (none) -> EXCLUDE
Changed lines of the file:
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@@
 <setting verticaltext="up"/>
 </settings>
-<grid distance="0.05" unitdist="inch" unit="inch" style="lines" multiple="1" display="no" altdistance="0.01" altunitdist="inch" altunit="inch"/>
+<grid distance="0.1" unitdist="inch" unit="inch" style="lines" multiple="1" display="no" altdistance="0.01" altunitdist="inch" altunit="inch"/>
 <layers>
 <layer number="1" name="Top" color="4" fill="1" visible="no" active="no"/>
@@
 </part>
 <part name="AGND27" library="supplies" deviceset="AGND" device=""/>
-<part name="TP1" library="test" deviceset="TESTPOINT-WITH-GND" device=""/>
-<part name="TP2" library="test" deviceset="TESTPOINT-WITH-GND" device=""/>
-<part name="TP3" library="test" deviceset="TESTPOINT-WITH-GND" device=""/>
+<part name="TP1" library="test" deviceset="TESTPOINT-WITH-GND" device="">
+<attribute name="BOM" value="EXCLUDE"/>
+</part>
+<part name="TP2" library="test" deviceset="TESTPOINT-WITH-GND" device="">
+<attribute name="BOM" value="EXCLUDE"/>
+</part>
+<part name="TP3" library="test" deviceset="TESTPOINT-WITH-GND" device="">
+<attribute name="BOM" value="EXCLUDE"/>
+</part>
 <part name="AGND28" library="supplies" deviceset="AGND" device=""/>
 <part name="+3V7" library="supplies" deviceset="+3V3" device=""/>
@@
 <attribute name="BOM" x="238.76" y="25.4" size="1.778" layer="96" display="off"/>
 </instance>
-<instance part="TP1" gate="G$1" x="201.93" y="63.5"/>
-<instance part="TP2" gate="G$1" x="201.93" y="46.99"/>
-<instance part="TP3" gate="G$1" x="201.93" y="30.48"/>
+<instance part="TP1" gate="G$1" x="201.93" y="63.5">
+<attribute name="BOM" x="201.93" y="63.5" size="1.778" layer="96" display="off"/>
+</instance>
+<instance part="TP2" gate="G$1" x="201.93" y="46.99">
+<attribute name="BOM" x="201.93" y="46.99" size="1.778" layer="96" display="off"/>
+</instance>
+<instance part="TP3" gate="G$1" x="201.93" y="30.48">
+<attribute name="BOM" x="201.93" y="30.48" size="1.778" layer="96" display="off"/>
+</instance>
 <instance part="AGND28" gate="VR1" x="191.77" y="16.51"/>
 <instance part="AGND12" gate="VR1" x="132.08" y="55.88"/>
@@
 </sheet>
 </sheets>
-<errors>
-</errors>
 </schematic>
 </drawing>

Commit message: BOM tweaks to account for supply chain issues.
Parts:
- D1: PN 598-8020-107F -> APT1608SURCK
- D3: PN 598-8081-107F -> 150060GS75000
- R13: PN RC0402FR-0727KL -> ERJ-2RKF2702X
- S1, S2: PN SKQGAKE010 -> SKQGADE010
Changed lines of the file:
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@@
 <part name="AGND10" library="supplies" deviceset="AGND" device=""/>
 <part name="D1" library="dialight" deviceset="DIALIGHT-598-MICROSMD" device="-0603" value="2V, 5mA">
-<attribute name="PN" value="598-8020-107F"/>
+<attribute name="PN" value="APT1608SURCK"/>
 </part>
 <part name="R4" library="passives" deviceset="RESISTOR-HORIZONTAL" device="-0603" value="330">
@@
 <part name="+3V3" library="supplies" deviceset="+3V3" device=""/>
 <part name="S1" library="switches" deviceset="MOMENTARY" device="-ALPS-SKQG" value="RESET">
-<attribute name="PN" value="SKQGAKE010"/>
+<attribute name="PN" value="SKQGADE010"/>
 </part>
 <part name="R7" library="passives" deviceset="RESISTOR" device="-0402" value="10K">
@@
 </part>
 <part name="S2" library="switches" deviceset="MOMENTARY" device="-ALPS-SKQG" value="UPLOAD">
-<attribute name="PN" value="SKQGAKE010"/>
+<attribute name="PN" value="SKQGADE010"/>
 </part>
 <part name="AGND17" library="supplies" deviceset="AGND" device=""/>
@@
 </part>
 <part name="R13" library="passives" deviceset="RESISTOR-HORIZONTAL" device="-0402" value="27K">
-<attribute name="PN" value="RC0402FR-0727KL"/>
+<attribute name="PN" value="ERJ-2RKF2702X"/>
 </part>
 <part name="R14" library="passives" deviceset="RESISTOR-HORIZONTAL" device="-0402" value="1M">
@@
 </part>
 <part name="D3" library="dialight" deviceset="DIALIGHT-598-MICROSMD" device="-0603" value="3.2V, 5mA">
-<attribute name="PN" value="598-8081-107F"/>
+<attribute name="PN" value="150060GS75000"/>
 </part>
 <part name="AGND27" library="supplies" deviceset="AGND" device=""/>

Commit message: A few fixes after testing the rev A1 boards.
Just fixing up a fix issues I found while build/testing the rev A1
boards, namely:
- using wrong footprint for T1/T2
- LEDs way too bright; adjusted series resistors
- used wrong part number for boost converter (ooof!)
- shoved HDMI connector closer to the edge
- added outlines to the various sections
- shuffled around test points and labels
Parts:
- removed TP3: TESTPOINT-WITH-GND, test:TESTPOINT-WITH-GND
- R16: value 330 -> 270; PN RC0603FR-07330RL -> RC0603FR-07270RL
- R4: value 330 -> 680; PN RC0603FR-07330RL -> RC0603FR-07680RL
- T1, T2: device transistors:BJT-NPN-SC-70 -> transistors:BJT-NPN-SOT-23
- U2: value TPS61200DRC -> TPS61201DRC; PN TPS61200DRCR -> TPS61201DRCR
Connections:
- net AGND: no longer TP3.G
- net VBAT: no longer TP3.S
Changed lines of the file:
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@@
 <attribute name="PN" value="MCP73831T-2ACI/OT"/>
 </part>
-<part name="U2" library="texas-instruments" deviceset="TPS6120" device="0DRC">
-<attribute name="PN" value="TPS61200DRCR"/>
+<part name="U2" library="texas-instruments" deviceset="TPS6120" device="0DRC" value="TPS61201DRC">
+<attribute name="PN" value="TPS61201DRCR"/>
 </part>
 <part name="C1" library="passives" deviceset="CAPACITOR" device="-0603" value="4.7uF">
@@
 <attribute name="PN" value="APT1608SURCK"/>
 </part>
-<part name="R4" library="passives" deviceset="RESISTOR-HORIZONTAL" device="-0603" value="330">
-<attribute name="PN" value="RC0603FR-07330RL"/>
+<part name="R4" library="passives" deviceset="RESISTOR-HORIZONTAL" device="-0603" value="680">
+<attribute name="PN" value="RC0603FR-07680RL"/>
 </part>
 <part name="AGND11" library="supplies" deviceset="AGND" device=""/>
@@
 <attribute name="BOM" value="EXCLUDE"/>
 </part>
-<part name="T1" library="transistors" deviceset="BJT-NPN" device="-SC-70" value="MMBT3904">
+<part name="T1" library="transistors" deviceset="BJT-NPN" device="-SOT-23" value="MMBT3904">
 <attribute name="PN" value="MMBT3904LT1G"/>
 </part>
-<part name="T2" library="transistors" deviceset="BJT-NPN" device="-SC-70" value="MMBT3904">
+<part name="T2" library="transistors" deviceset="BJT-NPN" device="-SOT-23" value="MMBT3904">
 <attribute name="PN" value="MMBT3904LT1G"/>
 </part>
@@
 <attribute name="BOM" value="EXCLUDE"/>
 </part>
-<part name="R16" library="passives" deviceset="RESISTOR-HORIZONTAL" device="-0603" value="330">
-<attribute name="PN" value="RC0603FR-07330RL"/>
+<part name="R16" library="passives" deviceset="RESISTOR-HORIZONTAL" device="-0603" value="270">
+<attribute name="PN" value="RC0603FR-07270RL"/>
 </part>
 <part name="D3" library="dialight" deviceset="DIALIGHT-598-MICROSMD" device="-0603" value="3.2V, 5mA">
@@
 </part>
 <part name="TP2" library="test" deviceset="TESTPOINT-WITH-GND" device="">
-<attribute name="BOM" value="EXCLUDE"/>
-</part>
-<part name="TP3" library="test" deviceset="TESTPOINT-WITH-GND" device="">
 <attribute name="BOM" value="EXCLUDE"/>
 </part>
@@
 <attribute name="BOM" x="201.93" y="46.99" size="1.778" layer="96" display="off"/>
 </instance>
-<instance part="TP3" gate="G$1" x="201.93" y="30.48">
-<attribute name="BOM" x="201.93" y="30.48" size="1.778" layer="96" display="off"/>
-</instance>
 <instance part="AGND28" gate="VR1" x="191.77" y="16.51"/>
 <instance part="AGND12" gate="VR1" x="132.08" y="55.88"/>
@@
 <pinref part="AGND28" gate="VR1" pin="AGND"/>
 <wire x1="191.77" y1="59.69" x2="191.77" y2="43.18" width="0.1524" layer="91"/>
-<pinref part="TP3" gate="G$1" pin="G"/>
-<wire x1="191.77" y1="43.18" x2="191.77" y2="26.67" width="0.1524" layer="91"/>
-<wire x1="191.77" y1="26.67" x2="191.77" y2="19.05" width="0.1524" layer="91"/>
-<wire x1="199.39" y1="26.67" x2="191.77" y2="26.67" width="0.1524" layer="91"/>
-<junction x="191.77" y="26.67"/>
+<wire x1="191.77" y1="43.18" x2="191.77" y2="19.05" width="0.1524" layer="91"/>
 <pinref part="TP2" gate="G$1" pin="G"/>
 <wire x1="199.39" y1="43.18" x2="191.77" y2="43.18" width="0.1524" layer="91"/>
@@
 <label x="130.81" y="68.58" size="2.54" layer="95" rot="R180" xref="yes"/>
 </segment>
-<segment>
-<pinref part="TP3" gate="G$1" pin="S"/>
-<wire x1="199.39" y1="30.48" x2="185.42" y2="30.48" width="0.1524" layer="91"/>
-<label x="185.42" y="30.48" size="2.54" layer="95" rot="R180" xref="yes"/>
-</segment>
-</net>
+</net>
